File: HARDWARE/TeR_ECU/TeR_ECU/CAN1.kicad_sch (KiCad schematic)
At the start: 7 parts, among them U1 SN65HVD230

Commit message: Micro
Changed lines of the file:
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@@
 (kicad_sch (version 20230121) (generator eeschema)
   (paper "A4")
-  (junction (at 139.7 101.6) (diameter 0) (color 0 0 0 0)
-  )
   (junction (at 93.98 96.52) (diameter 0) (color 0 0 0 0)
   )
@@
   (junction (at 173.99 85.09) (diameter 0) (color 0 0 0 0)
   )
-  (junction (at 139.7 69.85) (diameter 0) (color 0 0 0 0)
+  (junction (at 139.7 71.12) (diameter 0) (color 0 0 0 0)
   )
   (junction (at 179.07 87.63) (diameter 0) (color 0 0 0 0)
   )
+  (junction (at 139.7 100.33) (diameter 0) (color 0 0 0 0)
+  )
   (junction (at 93.98 73.66) (diameter 0) (color 0 0 0 0)
   )
-  (wire (pts (xy 109.22 69.85) (xy 139.7 69.85))
+  (wire (pts (xy 109.22 71.12) (xy 139.7 71.12))
     (stroke (width 0) (type default))
   )
@@
     (stroke (width 0) (type default))
   )
-  (wire (pts (xy 139.7 69.85) (xy 139.7 72.39))
+  (wire (pts (xy 139.7 71.12) (xy 139.7 72.39))
     (stroke (width 0) (type default))
   )
@@
     (stroke (width 0) (type default))
   )
-  (wire (pts (xy 139.7 69.85) (xy 163.83 69.85))
+  (wire (pts (xy 139.7 71.12) (xy 163.83 71.12))
     (stroke (width 0) (type default))
   )
@@
     (stroke (width 0) (type default))
   )
-  (wire (pts (xy 139.7 101.6) (xy 163.83 101.6))
+  (wire (pts (xy 139.7 100.33) (xy 163.83 100.33))
     (stroke (width 0) (type default))
   )
@@
     (stroke (width 0) (type default))
   )
-  (wire (pts (xy 109.22 101.6) (xy 139.7 101.6))
+  (wire (pts (xy 109.22 100.33) (xy 139.7 100.33))
     (stroke (width 0) (type default))
   )
@@
     (stroke (width 0) (type default))
   )
-  (wire (pts (xy 139.7 101.6) (xy 139.7 97.79))
-    (stroke (width 0) (type default))
-  )
   (wire (pts (xy 134.62 85.09) (xy 134.62 80.01))
     (stroke (width 0) (type default))
   )
-  (wire (pts (xy 109.22 85.09) (xy 109.22 69.85))
+  (wire (pts (xy 109.22 85.09) (xy 109.22 71.12))
     (stroke (width 0) (type default))
   )
@@
     (stroke (width 0) (type default))
   )
-  (wire (pts (xy 163.83 69.85) (xy 163.83 85.09))
+  (wire (pts (xy 139.7 100.33) (xy 139.7 97.79))
+    (stroke (width 0) (type default))
+  )
+  (wire (pts (xy 163.83 71.12) (xy 163.83 85.09))
     (stroke (width 0) (type default))
   )
@@
     (stroke (width 0) (type default))
   )
-  (wire (pts (xy 109.22 87.63) (xy 109.22 101.6))
+  (wire (pts (xy 109.22 87.63) (xy 109.22 100.33))
     (stroke (width 0) (type default))
   )
-  (wire (pts (xy 163.83 87.63) (xy 163.83 101.6))
+  (wire (pts (xy 163.83 87.63) (xy 163.83 100.33))
     (stroke (width 0) (type default))
   )
