File: HARDWARE/TeR_ECU/TeR_ECU/Deteccion_señales.kicad_sch (KiCad schematic)
At the start: 4 parts

Commit message: Listo para empezar con layout
Parts:
- R10, R11, R12, R9: footprint (none) -> Resistor_SMD:R_0805_2012Metric
Changed lines of the file:
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@@
       (effects (font (size 1.27 1.27)) (justify left))
     )
-    (property "Footprint" "" (at 120.142 72.39 90)
+    (property "Footprint" "Resistor_SMD:R_0805_2012Metric" (at 120.142 72.39 90)
       (effects (font (size 1.27 1.27)) hide)
     )
@@
       (effects (font (size 1.27 1.27)) (justify left))
     )
-    (property "Footprint" "" (at 163.322 87.63 90)
+    (property "Footprint" "Resistor_SMD:R_0805_2012Metric" (at 163.322 87.63 90)
       (effects (font (size 1.27 1.27)) hide)
     )
@@
       (effects (font (size 1.27 1.27)) (justify left))
     )
-    (property "Footprint" "" (at 163.322 72.39 90)
+    (property "Footprint" "Resistor_SMD:R_0805_2012Metric" (at 163.322 72.39 90)
       (effects (font (size 1.27 1.27)) hide)
     )
@@
       (effects (font (size 1.27 1.27)) (justify left))
     )
-    (property "Footprint" "" (at 120.142 87.63 90)
+    (property "Footprint" "Resistor_SMD:R_0805_2012Metric" (at 120.142 87.63 90)
       (effects (font (size 1.27 1.27)) hide)
     )
