File: HARDWARE/TeR_ECU/TeR_ECU/Functions.kicad_sch (KiCad schematic)
At the start: 7 parts, among them Q1 ZXMN3F30FH, Q2 ZXMN3F30FH

Commit message: Listo para empezar con layout
Parts:
- R13, R14, R15, R16, R17: footprint (none) -> Resistor_SMD:R_0805_2012Metric
Changed lines of the file:
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@@
       (effects (font (size 1.27 1.27)))
     )
-    (property "Footprint" "" (at 83.82 70.612 90)
+    (property "Footprint" "Resistor_SMD:R_0805_2012Metric" (at 83.82 70.612 90)
       (effects (font (size 1.27 1.27)) hide)
     )
@@
       (effects (font (size 1.27 1.27)) (justify left))
     )
-    (property "Footprint" "" (at 150.622 76.2 90)
+    (property "Footprint" "Resistor_SMD:R_0805_2012Metric" (at 150.622 76.2 90)
       (effects (font (size 1.27 1.27)) hide)
     )
@@
       (effects (font (size 1.27 1.27)))
     )
-    (property "Footprint" "" (at 160.02 68.072 90)
+    (property "Footprint" "Resistor_SMD:R_0805_2012Metric" (at 160.02 68.072 90)
       (effects (font (size 1.27 1.27)) hide)
     )
@@
       (effects (font (size 1.27 1.27)) (justify right))
     )
-    (property "Footprint" "" (at 187.198 54.61 90)
+    (property "Footprint" "Resistor_SMD:R_0805_2012Metric" (at 187.198 54.61 90)
       (effects (font (size 1.27 1.27)) hide)
     )
@@
       (effects (font (size 1.27 1.27)) (justify right))
     )
-    (property "Footprint" "" (at 201.168 54.61 90)
+    (property "Footprint" "Resistor_SMD:R_0805_2012Metric" (at 201.168 54.61 90)
       (effects (font (size 1.27 1.27)) hide)
     )
