File: HARDWARE/TeR_ECU/TeR_ECU/POWER.kicad_sch (KiCad schematic)
At the start: 13 parts, among them U2 TSR_1-2450, U3 LM1117MP-3.3, U4 TSR_1-24120

Commit message: Listo para empezar con layout
Connections:
- net +5V: no longer U4.3 (Vout)
- new net +12V: U4.3 (Vout)
Changed lines of the file:
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@@
       (project "TeR_ECU"
         (path "/84413845-c4f3-4743-bcd2-a67649c90902/b76a95f3-584c-4daf-bbe9-70945b593e94"
-          (reference "U2") (unit 1)
+          (reference "U5") (unit 1)
+        )
+      )
+    )
+  )
+  (symbol (lib_id "power:+12V") (at 113.03 82.55 0) (unit 1)
+    (in_bom yes) (on_board yes) (dnp no) (fields_autoplaced)
+    (property "Reference" "#PWR042" (at 113.03 86.36 0)
+      (effects (font (size 1.27 1.27)) hide)
+    )
+    (property "Value" "+12V" (at 113.03 77.47 0)
+      (effects (font (size 1.27 1.27)))
+    )
+    (property "Footprint" "" (at 113.03 82.55 0)
+      (effects (font (size 1.27 1.27)) hide)
+    )
+    (property "Datasheet" "" (at 113.03 82.55 0)
+      (effects (font (size 1.27 1.27)) hide)
+    )
+    (pin "1")
+    (instances
+      (project "TeR_ECU"
+        (path "/84413845-c4f3-4743-bcd2-a67649c90902/b76a95f3-584c-4daf-bbe9-70945b593e94"
+          (reference "#PWR042") (unit 1)
         )
       )
@@
       (project "TeR_ECU"
         (path "/84413845-c4f3-4743-bcd2-a67649c90902/b76a95f3-584c-4daf-bbe9-70945b593e94"
-          (reference "C12") (unit 1)
+          (reference "C20") (unit 1)
         )
       )
@@
       (project "TeR_ECU"
         (path "/84413845-c4f3-4743-bcd2-a67649c90902/b76a95f3-584c-4daf-bbe9-70945b593e94"
-          (reference "C13") (unit 1)
+          (reference "C21") (unit 1)
         )
       )
@@
       (project "TeR_ECU"
         (path "/84413845-c4f3-4743-bcd2-a67649c90902/b76a95f3-584c-4daf-bbe9-70945b593e94"
-          (reference "C18") (unit 1)
+          (reference "C19") (unit 1)
         )
       )
@@
       (project "TeR_ECU"
         (path "/84413845-c4f3-4743-bcd2-a67649c90902/b76a95f3-584c-4daf-bbe9-70945b593e94"
-          (reference "C9") (unit 1)
+          (reference "C16") (unit 1)
         )
       )
@@
       (project "TeR_ECU"
         (path "/84413845-c4f3-4743-bcd2-a67649c90902/b76a95f3-584c-4daf-bbe9-70945b593e94"
-          (reference "C17") (unit 1)
+          (reference "C18") (unit 1)
         )
       )
@@
       (project "TeR_ECU"
         (path "/84413845-c4f3-4743-bcd2-a67649c90902/b76a95f3-584c-4daf-bbe9-70945b593e94"
-          (reference "C10") (unit 1)
+          (reference "C17") (unit 1)
         )
       )
@@
       (project "TeR_ECU"
         (path "/84413845-c4f3-4743-bcd2-a67649c90902/b76a95f3-584c-4daf-bbe9-70945b593e94"
-          (reference "U3") (unit 1)
+          (reference "U6") (unit 1)
         )
       )
@@
         )
       )
-    )
-  )
-  (symbol (lib_id "power:+5V") (at 113.03 82.55 0) (unit 1)
-    (in_bom yes) (on_board yes) (dnp no) (fields_autoplaced)
-    (property "Reference" "#PWR016" (at 113.03 86.36 0)
-      (effects (font (size 1.27 1.27)) hide)
-    )
-    (property "Value" "+5V" (at 113.03 78.74 0)
-      (effects (font (size 1.27 1.27)))
-    )
-    (property "Footprint" "" (at 113.03 82.55 0)
-      (effects (font (size 1.27 1.27)) hide)
-    )
-    (property "Datasheet" "" (at 113.03 82.55 0)
-      (effects (font (size 1.27 1.27)) hide)
-    )
-    (pin "1")
-    (instances
-      (project "TER_PEDAL"
-        (path "/73ede3a3-6344-40fe-9207-10ff50d388ba/6f10bd65-583f-4818-aeb8-8b5e6e37f336"
-          (reference "#PWR016") (unit 1)
-        )
-      )
-      (project "TeR_ECU"
-        (path "/84413845-c4f3-4743-bcd2-a67649c90902/b76a95f3-584c-4daf-bbe9-70945b593e94"
-          (reference "#PWR042") (unit 1)
-        )
-      )
