File: HARDWARE/TeR_ECU/TeR_ECU/CAN.kicad_sch (KiCad schematic)
At the start: 7 parts, among them U1 SN65HVD230

Commit message: Falta conector tocho
Parts:
- C3: value C -> 4.7nF; footprint (none) -> Capacitor_SMD:C_0603_1608Metric
- JP1: footprint (none) -> Jumper:SolderJumper-3_P1.3mm_Open_Pad1.0x1.5mm
- R1, R2: value R -> 60R
Changed lines of the file:
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@@
       (effects (font (size 1.27 1.27)) (justify left))
     )
-    (property "Value" "R" (at 142.24 77.47 0)
+    (property "Value" "60R" (at 142.24 77.47 0)
       (effects (font (size 1.27 1.27)) (justify left))
     )
@@
       (effects (font (size 1.27 1.27)) (justify left))
     )
-    (property "Value" "R" (at 142.24 95.25 0)
+    (property "Value" "60R" (at 142.24 95.25 0)
       (effects (font (size 1.27 1.27)) (justify left))
     )
@@
       (effects (font (size 1.27 1.27)))
     )
-    (property "Value" "C" (at 124.46 80.01 90)
-      (effects (font (size 1.27 1.27)))
-    )
-    (property "Footprint" "" (at 120.65 86.0552 0)
+    (property "Value" "4.7nF" (at 124.46 80.01 90)
+      (effects (font (size 1.27 1.27)))
+    )
+    (property "Footprint" "Capacitor_SMD:C_0603_1608Metric" (at 120.65 86.0552 0)
       (effects (font (size 1.27 1.27)) hide)
     )
@@
       (effects (font (size 1.27 1.27)) (justify left))
     )
-    (property "Footprint" "" (at 139.7 85.09 0)
-      (effects (font (size 1.27 1.27)) hide)
-    )
+    (property "Footprint" "Jumper:SolderJumper-3_P1.3mm_Open_Pad1.0x1.5mm" (at 139.7 85.09 0)
+      (effects (font (size 1.27 1.27)) hide)
+    )

Commit message: Listo para empezar con layout
Parts:
- R1, R2: footprint (none) -> Resistor_SMD:R_0805_2012Metric
Changed lines of the file:
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@@
       (effects (font (size 1.27 1.27)) (justify left))
     )
-    (property "Footprint" "" (at 137.922 76.2 90)
+    (property "Footprint" "Resistor_SMD:R_0805_2012Metric" (at 137.922 76.2 90)
       (effects (font (size 1.27 1.27)) hide)
     )
@@
       (effects (font (size 1.27 1.27)) (justify left))
     )
-    (property "Footprint" "" (at 137.922 93.98 90)
+    (property "Footprint" "Resistor_SMD:R_0805_2012Metric" (at 137.922 93.98 90)
       (effects (font (size 1.27 1.27)) hide)
     )

Commit message: Revisar y empezar Layout
Parts:
- R1, R2: value 60R -> 50R
Other:
- note added: "Valorar leds de estado de las lineas TX y RX"
Changed lines of the file:
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@@
     (stroke (width 0) (type default))
+  )
+  (text "Valorar leds de estado de las lineas TX y RX" (at 52.07 49.53 0)
+    (effects (font (size 1.27 1.27)) (justify left bottom))
   )
   (text "High speed mode\n" (at 78.74 99.06 0)
@@
       (effects (font (size 1.27 1.27)) (justify left))
     )
-    (property "Value" "60R" (at 142.24 77.47 0)
+    (property "Value" "50R" (at 142.24 77.47 0)
       (effects (font (size 1.27 1.27)) (justify left))
     )
@@
       (effects (font (size 1.27 1.27)) (justify left))
     )
-    (property "Value" "60R" (at 142.24 95.25 0)
+    (property "Value" "50R" (at 142.24 95.25 0)
       (effects (font (size 1.27 1.27)) (justify left))
     )
