File: HARDWARE/TeR_ECU/TeR_ECU/Micro.kicad_sch (KiCad schematic)
At the start: 1 part, among them U3 STM32F446RETx

Commit message: Micro
Parts:
- added C10: 10nF, Capacitor_SMD:C_0805_2012Metric, symbol Device:C
- added C11, C12: 1uF, Capacitor_SMD:C_0805_2012Metric, symbol Device:C
- added C13, C6, C7, C8, C9: 100nF, Capacitor_SMD:C_0805_2012Metric, symbol Device:C
- added C5: 10uF, Capacitor_SMD:C_0805_2012Metric, symbol Device:C
- added FB1: 120R, symbol Device:FerriteBead
- added JP1: BOOT0, symbol Jumper:Jumper_3_Bridged12
- added JP2: BOOT1, symbol Jumper:Jumper_3_Bridged12
- added R5: 100R, symbol Device:R
- added R6, R7: 10k, symbol Device:R
- added SW1: RST, symbol Switch:SW_SPST
Connections:
- net +3.3V: now reaches U3.1 (VBAT)
- net +3.3V: now also U3.19 (VDD), U3.32 (VDD), U3.48 (VDD), U3.64 (VDD), C12.2, C5.2, C6.2, C7.2, C8.2, C9.2, FB1.2, JP1.3 (B), JP2.3 (B)
- net GND: now reaches U3.12 (VSSA)
- net GND: now also U3.18 (VSS), U3.31 (VSS), U3.47 (VSS), U3.63 (VSS), C10.1, C11.1, C12.1, C13.1, C5.1, C6.1, C7.1, C8.1, C9.1, JP1.1 (A), JP2.1 (A), SW1.1 (A)
- net +3.3VADC: now reaches U3.13 (VDDA)
- net +3.3VADC: now also C10.2, C11.2, FB1.1
- net BOOT1: now reaches U3.28 (PB2)
- net BOOT1: now also R7.2
- net BOOT0: now reaches U3.60 (BOOT0)
- net BOOT0: now also R6.2
- net NRST: now reaches U3.7 (NRST)
- net NRST: now also C13.2, R5.2
- new net: JP1.2 (C), R6.1
- new net: R5.1, SW1.2 (B)
- new net: JP2.2 (C), R7.1
Other:
- note added: "ADC Filter"
- note added: "BOOT Selector"
- note added: "PSU Decoupling"
- note added: "Place each next to each Vdd pin"
- note added: "Reset Button"
- moved on the sheet: U3

Commit message: Esquematico Micro para revisar
Parts:
- added C14, C15: 10pF, Capacitor_SMD:C_0805_2012Metric, symbol Device:C
- added J4: Debug, Connector_PinHeader_2.00mm:PinHeader_1x04_P2.00mm_Vertical, symbol Connector:Conn_01x04_Pin
- added R8: 300R, symbol Device:R
- added Y1: Crystal, symbol Device:Crystal
- renumbered JP1 to JP3, JP2 to JP4
Connections:
- net +3.3V: now also J4.4 (Pin_4)
- net GND: now also C14.2, C15.1, J4.1 (Pin_1)
- net SWDIO: now reaches U3.46 (PA13)
- net SWDIO: now also J4.2 (Pin_2)
- net SWCLK: now reaches U3.49 (PA14)
- net SWCLK: now also J4.3 (Pin_3)
- net OSC_IN: now reaches U3.5 (PH0)
- net OSC_IN: now also C14.1, Y1.1
- net OSC_OUT: now reaches U3.6 (PH1)
- net OSC_OUT: now also R8.1
- new net: C15.2, R8.2, Y1.2
Other:
- note added: "CL = (Cl1 * CL2) / (CL1+CL2)"
- note added: "Debug Connector"
- note added: "HSE OSCILATOR"
- note added: "Rext = 60Ω * 5 = 300Ω"
- note added: "XRCGB32M000F2N13R0 (Propuesta, vale cualquiera,calculos)"

Commit message: Menos el del conector grande, los demas esquematicos acabados
Parts:
- added C16: 100nF, Capacitor_SMD:C_0805_2012Metric, symbol Device:C
Connections:
- net +3.3V: now also C16.2
- net GND: now also C16.1
- net CAN2_RX: now reaches U3.33 (PB12)
- net CAN2_TX: now reaches U3.34 (PB13)
- net BSPD_3V3: now reaches U3.39 (PC8)
- net TSMS_3V3: now reaches U3.40 (PC9)
- net CAN1_RX: now reaches U3.44 (PA11)
- net CAN1_TX: now reaches U3.45 (PA12)
- net BL: now reaches U3.52 (PC11)
- net Horn: now reaches U3.53 (PC12)
Other:
- moved on the sheet: C10, C11, C12, C13, C14, C15, C5, C6, C7, C8, C9, FB1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

Commit message: Falta conector tocho
Parts:
- C10, C11, C12: footprint Capacitor_SMD:C_0805_2012Metric -> Capacitor_SMD:C_0402_1005Metric_Pad0.74x0.62mm_HandSolder
- C13, C14, C15: footprint Capacitor_SMD:C_0805_2012Metric -> Capacitor_SMD:C_0603_1608Metric
- FB1: footprint (none) -> Inductor_SMD:L_0805_2012Metric
- JP3, JP4: footprint (none) -> Connector_PinHeader_2.00mm:PinHeader_1x03_P2.00mm_Vertical
- R5, R6, R7: footprint (none) -> Resistor_SMD:R_0603_1608Metric
- R8: footprint (none) -> Resistor_SMD:R_0402_1005Metric
- SW1: footprint (none) -> Button_Switch_SMD:SW_Tactile_SPST_NO_Straight_CK_PTS636Sx25SMTRLFS
- Y1: footprint (none) -> Crystal:Crystal_SMD_5032-2Pin_5.0x3.2mm
Other:
- moved on the sheet: R8
Changed lines of the file:
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@@
+    (stroke (width 0) (type default))
+  )
+  (wire (pts (xy 45.72 88.9) (xy 58.42 88.9))
+    (stroke (width 0) (type default))
+  )
+  (wire (pts (xy 124.46 68.58) (xy 134.62 68.58))
+    (stroke (width 0) (type default))
+  )
+  (wire (pts (xy 29.21 147.32) (xy 36.83 147.32))
+    (stroke (width 0) (type default))
+  )
+  (wire (pts (xy 54.61 24.13) (xy 64.77 24.13))
+    (stroke (width 0) (type default))
+  )
+  (polyline (pts (xy 251.46 49.53) (xy 284.48 49.53))
+    (stroke (width 0) (type default))
+  )
+  (wire (pts (xy 55.88 67.31) (xy 55.88 69.85))
+    (stroke (width 0) (type default))
+  )
+  (wire (pts (xy 124.46 101.6) (xy 134.62 101.6))
+    (stroke (width 0) (type default))
+  )
+  (wire (pts (xy 154.94 142.24) (xy 154.94 143.51))
+    (stroke (width 0) (type default))
+  )
+  (wire (pts (xy 124.46 66.04) (xy 134.62 66.04))
+    (stroke (width 0) (type default))
+  )
+  (wire (pts (xy 21.59 130.81) (xy 21.59 128.27))
+    (stroke (width 0) (type default))
+  )
+  (wire (pts (xy 50.8 57.15) (xy 55.88 57.15))
+    (stroke (width 0) (type default))
+  )
+  (wire (pts (xy 24.13 57.15) (xy 35.56 57.15))
+    (stroke (width 0) (type default))
+  )
+  (polyline (pts (xy 74.93 111.76) (xy 74.93 149.86))
+    (stroke (width 0) (type default))
+  )
+  (wire (pts (xy 24.13 59.69) (xy 24.13 57.15))
+    (stroke (width 0) (type default))
+  )
+  (wire (pts (xy 55.88 55.88) (xy 55.88 57.15))
+    (stroke (width 0) (type default))
+  )
+  (polyline (pts (xy 12.7 149.86) (xy 74.93 149.86))
+    (stroke (width 0) (type default))
+  )
+  (wire (pts (xy 27.94 88.9) (xy 31.75 88.9))
+    (stroke (width 0) (type default))
+  )
+  (wire (pts (xy 152.4 143.51) (xy 152.4 144.78))
+    (stroke (width 0) (type default))
+  )
+  (wire (pts (xy 44.45 31.75) (xy 54.61 31.75))
     (stroke (width 0) (type default))
   )
@@
     (stroke (width 0) (type default))
   )
-  (wire (pts (xy 45.72 88.9) (xy 58.42 88.9))
-    (stroke (width 0) (type default))
-  )
-  (wire (pts (xy 124.46 68.58) (xy 134.62 68.58))
-    (stroke (width 0) (type default))
-  )
-  (wire (pts (xy 29.21 147.32) (xy 36.83 147.32))
-    (stroke (width 0) (type default))
-  )
-  (wire (pts (xy 54.61 24.13) (xy 64.77 24.13))
-    (stroke (width 0) (type default))
-  )
-  (polyline (pts (xy 251.46 49.53) (xy 284.48 49.53))
-    (stroke (width 0) (type default))
-  )
-  (wire (pts (xy 55.88 67.31) (xy 55.88 69.85))
-    (stroke (width 0) (type default))
-  )
-  (wire (pts (xy 124.46 101.6) (xy 134.62 101.6))
-    (stroke (width 0) (type default))
-  )
-  (wire (pts (xy 154.94 142.24) (xy 154.94 143.51))
-    (stroke (width 0) (type default))
-  )
-  (wire (pts (xy 124.46 66.04) (xy 134.62 66.04))
-    (stroke (width 0) (type default))
-  )
-  (wire (pts (xy 21.59 130.81) (xy 21.59 128.27))
-    (stroke (width 0) (type default))
-  )
-  (wire (pts (xy 50.8 57.15) (xy 55.88 57.15))
-    (stroke (width 0) (type default))
-  )
-  (wire (pts (xy 24.13 57.15) (xy 35.56 57.15))
-    (stroke (width 0) (type default))
-  )
-  (polyline (pts (xy 74.93 111.76) (xy 74.93 149.86))
-    (stroke (width 0) (type default))
-  )
-  (wire (pts (xy 24.13 59.69) (xy 24.13 57.15))
-    (stroke (width 0) (type default))
-  )
-  (wire (pts (xy 55.88 55.88) (xy 55.88 57.15))
-    (stroke (width 0) (type default))
-  )
-  (polyline (pts (xy 12.7 149.86) (xy 74.93 149.86))
-    (stroke (width 0) (type default))
-  )
-  (wire (pts (xy 27.94 88.9) (xy 31.75 88.9))
-    (stroke (width 0) (type default))
-  )
-  (wire (pts (xy 152.4 143.51) (xy 152.4 144.78))
-    (stroke (width 0) (type default))
-  )
-  (wire (pts (xy 44.45 31.75) (xy 54.61 31.75))
-    (stroke (width 0) (type default))
-  )
   (polyline (pts (xy 12.7 77.47) (xy 74.93 77.47))
     (stroke (width 0) (type default))
@@
     (stroke (width 0) (type default))
   )
-  (wire (pts (xy 48.26 168.91) (xy 48.26 173.99))
+  (wire (pts (xy 48.26 170.18) (xy 48.26 173.99))
     (stroke (width 0) (type default))
   )
@@
   )
   (wire (pts (xy 124.46 99.06) (xy 134.62 99.06))
+    (stroke (width 0) (type default))
+  )
+  (wire (pts (xy 48.26 161.29) (xy 48.26 162.56))
     (stroke (width 0) (type default))
   )
@@
       (effects (font (size 1.27 1.27)) (justify right))
     )
-    (property "Footprint" "Capacitor_SMD:C_0805_2012Metric" (at 54.9148 59.69 0)
+    (property "Footprint" "Capacitor_SMD:C_0402_1005Metric_Pad0.74x0.62mm_HandSolder" (at 54.9148 59.69 0)
       (effects (font (size 1.27 1.27)) hide)
     )
@@
       (effects (font (size 1.27 1.27)) (justify right))
     )
-    (property "Footprint" "Capacitor_SMD:C_0805_2012Metric" (at 23.1648 59.69 0)
+    (property "Footprint" "Capacitor_SMD:C_0402_1005Metric_Pad0.74x0.62mm_HandSolder" (at 23.1648 59.69 0)
       (effects (font (size 1.27 1.27)) hide)
     )
@@
       (effects (font (size 1.27 1.27)) (justify right))
     )
-    (property "Footprint" "Capacitor_SMD:C_0805_2012Metric" (at 52.07 174.9552 0)
+    (property "Footprint" "Capacitor_SMD:C_0603_1608Metric" (at 52.07 174.9552 0)
       (effects (font (size 1.27 1.27)) hide)
     )
@@
       (effects (font (size 1.27 1.27)))
     )
-    (property "Footprint" "" (at 29.21 128.27 0)
+    (property "Footprint" "Connector_PinHeader_2.00mm:PinHeader_1x03_P2.00mm_Vertical" (at 29.21 128.27 0)
       (effects (font (size 1.27 1.27)) hide)
     )
@@
       (effects (font (size 1.27 1.27)) (justify left))
     )
-    (property "Footprint" "" (at 27.432 138.43 90)
+    (property "Footprint" "Resistor_SMD:R_0603_1608Metric" (at 27.432 138.43 90)
       (effects (font (size 1.27 1.27)) hide)
     )
@@
       (effects (font (size 1.27 1.27)))
     )
-    (property "Footprint" "" (at 35.56 90.678 90)
+    (property "Footprint" "Resistor_SMD:R_0603_1608Metric" (at 35.56 90.678 90)
       (effects (font (size 1.27 1.27)) hide)
     )
@@
       (effects (font (size 1.27 1.27)) (justify right))
     )
-    (property "Footprint" "Capacitor_SMD:C_0805_2012Metric" (at 44.7548 92.71 0)
+    (property "Footprint" "Capacitor_SMD:C_0603_1608Metric" (at 44.7548 92.71 0)
       (effects (font (size 1.27 1.27)) hide)
     )
@@
       (effects (font (size 1.27 1.27)) (justify left))
     )
-    (property "Footprint" "" (at 50.292 138.43 90)
+    (property "Footprint" "Resistor_SMD:R_0603_1608Metric" (at 50.292 138.43 90)
       (effects (font (size 1.27 1.27)) hide)
     )
@@
     )
   )
-  (symbol (lib_id "Device:R") (at 48.26 165.1 0) (unit 1)
-    (in_bom yes) (on_board yes) (dnp no) (fields_autoplaced)
-    (property "Reference" "R8" (at 50.8 163.83 0)
+  (symbol (lib_id "Device:R") (at 48.26 166.37 0) (unit 1)
+    (in_bom yes) (on_board yes) (dnp no) (fields_autoplaced)
+    (property "Reference" "R8" (at 50.8 165.1 0)
       (effects (font (size 1.27 1.27)) (justify left))
     )
-    (property "Value" "300R" (at 50.8 166.37 0)
+    (property "Value" "300R" (at 50.8 167.64 0)
       (effects (font (size 1.27 1.27)) (justify left))
     )
-    (property "Footprint" "" (at 46.482 165.1 90)
-      (effects (font (size 1.27 1.27)) hide)
-    )
-    (property "Datasheet" "~" (at 48.26 165.1 0)
+    (property "Footprint" "Resistor_SMD:R_0402_1005Metric" (at 46.482 166.37 90)
+      (effects (font (size 1.27 1.27)) hide)
+    )
+    (property "Datasheet" "~" (at 48.26 166.37 0)
       (effects (font (size 1.27 1.27)) hide)
     )
@@
       (effects (font (size 1.27 1.27)))
     )
-    (property "Footprint" "" (at 46.99 58.928 90)
+    (property "Footprint" "Inductor_SMD:L_0805_2012Metric" (at 46.99 58.928 90)
       (effects (font (size 1.27 1.27)) hide)
     )
@@
       (effects (font (size 1.27 1.27)) (justify right))
     )
-    (property "Footprint" "" (at 27.94 96.52 0)
+    (property "Footprint" "Button_Switch_SMD:SW_Tactile_SPST_NO_Straight_CK_PTS636Sx25SMTRLFS" (at 27.94 96.52 0)
       (effects (font (size 1.27 1.27)) hide)
     )
@@
       (effects (font (size 1.27 1.27)))
     )
-    (property "Footprint" "" (at 52.07 128.27 0)
+    (property "Footprint" "Connector_PinHeader_2.00mm:PinHeader_1x03_P2.00mm_Vertical" (at 52.07 128.27 0)
       (effects (font (size 1.27 1.27)) hide)
     )
@@
       (effects (font (size 1.27 1.27)))
     )
-    (property "Footprint" "" (at 41.91 173.99 0)
+    (property "Footprint" "Crystal:Crystal_SMD_5032-2Pin_5.0x3.2mm" (at 41.91 173.99 0)
       (effects (font (size 1.27 1.27)) hide)
     )
@@
       (effects (font (size 1.27 1.27)) (justify right))
     )
-    (property "Footprint" "Capacitor_SMD:C_0805_2012Metric" (at 34.5948 59.69 0)
+    (property "Footprint" "Capacitor_SMD:C_0402_1005Metric_Pad0.74x0.62mm_HandSolder" (at 34.5948 59.69 0)
       (effects (font (size 1.27 1.27)) hide)
     )
@@
       (effects (font (size 1.27 1.27)) (justify right))
     )
-    (property "Footprint" "Capacitor_SMD:C_0805_2012Metric" (at 25.4 174.9552 0)
-      (effects (font (size 1.27 1.27)) hide)
-    )
+    (property "Footprint" "Capacitor_SMD:C_0603_1608Metric" (at 25.4 174.9552 0)
+      (effects (font (size 1.27 1.27)) hide)
+    )

Commit message: Listo para empezar con layout
Connections:
- net IMP_LED: now reaches U3.20 (PA4)
- net DBG_LED: now reaches U3.21 (PA5)
- no-connect marks 0 -> 36
Changed lines of the file:
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@@
   (junction (at 34.29 24.13) (diameter 0) (color 0 0 0 0)
   )
+  (no_connect (at 134.62 83.82))
+  (no_connect (at 170.18 134.62))
+  (no_connect (at 170.18 114.3))
+  (no_connect (at 170.18 119.38))
+  (no_connect (at 134.62 80.01))
+  (no_connect (at 134.62 78.74))
+  (no_connect (at 170.18 81.28))
+  (no_connect (at 134.62 114.3))
+  (no_connect (at 170.18 55.88))
+  (no_connect (at 134.62 91.44))
+  (no_connect (at 170.18 93.98))
+  (no_connect (at 170.18 73.66))
+  (no_connect (at 134.62 121.92))
+  (no_connect (at 170.18 124.46))
+  (no_connect (at 170.18 63.5))
+  (no_connect (at 170.18 111.76))
+  (no_connect (at 170.18 60.96))
+  (no_connect (at 170.18 109.22))
+  (no_connect (at 170.18 106.68))
+  (no_connect (at 134.62 93.98))
+  (no_connect (at 170.18 132.08))
+  (no_connect (at 170.18 76.2))
+  (no_connect (at 170.18 120.65))
+  (no_connect (at 170.18 101.6))
+  (no_connect (at 134.62 111.76))
+  (no_connect (at 134.62 104.14))
+  (no_connect (at 134.62 96.52))
+  (no_connect (at 170.18 99.06))
+  (no_connect (at 134.62 73.66))
+  (no_connect (at 134.62 88.9))
+  (no_connect (at 170.18 116.84))
+  (no_connect (at 170.18 58.42))
+  (no_connect (at 170.18 71.12))
+  (no_connect (at 170.18 78.74))
+  (no_connect (at 134.62 86.36))
+  (no_connect (at 134.62 116.84))
   (wire (pts (xy 152.4 46.99) (xy 149.86 46.99))
     (stroke (width 0) (type default))
@@
     (stroke (width 0) (type default))
   )
+  (wire (pts (xy 170.18 66.04) (xy 177.8 66.04))
+    (stroke (width 0) (type default))
+  )
   (wire (pts (xy 124.46 68.58) (xy 134.62 68.58))
     (stroke (width 0) (type default))
@@
   )
   (wire (pts (xy 38.1 128.27) (xy 38.1 127))
+    (stroke (width 0) (type default))
+  )
+  (wire (pts (xy 170.18 68.58) (xy 177.8 68.58))
     (stroke (width 0) (type default))
   )
@@
     (effects (font (size 1.27 1.27)) (justify right))
   )
+  (hierarchical_label "IMP_LED" (shape input) (at 177.8 66.04 0) (fields_autoplaced)
+    (effects (font (size 1.27 1.27)) (justify left))
+  )
   (hierarchical_label "CAN2_RX" (shape input) (at 177.8 127 0) (fields_autoplaced)
     (effects (font (size 1.27 1.27)) (justify left))
@@
     (effects (font (size 1.27 1.27)) (justify left))
   )
+  (hierarchical_label "DBG_LED" (shape input) (at 177.8 68.58 0) (fields_autoplaced)
+    (effects (font (size 1.27 1.27)) (justify left))
+  )

Commit message: Revisar y empezar Layout
Connections:
- net LEDs: now reaches U3.38 (PC7)
- no-connect marks 36 -> 35
Changed lines of the file:
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@@
   (no_connect (at 134.62 111.76))
   (no_connect (at 134.62 104.14))
-  (no_connect (at 134.62 96.52))
   (no_connect (at 170.18 99.06))
   (no_connect (at 134.62 73.66))
@@
     (stroke (width 0) (type default))
   )
+  (wire (pts (xy 124.46 96.52) (xy 134.62 96.52))
+    (stroke (width 0) (type default))
+  )
   (wire (pts (xy 24.13 31.75) (xy 34.29 31.75))
     (stroke (width 0) (type default))
@@
     (effects (font (size 1.27 1.27)) (justify left))
   )
+  (hierarchical_label "LEDs" (shape output) (at 124.46 96.52 180) (fields_autoplaced)
+    (effects (font (size 1.27 1.27)) (justify right))
+  )
   (hierarchical_label "TSMS_3V3" (shape input) (at 124.46 101.6 180) (fields_autoplaced)

Commit message: Revisar y empezar Layout
Changed lines of the file:
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@@
     (effects (font (size 1.27 1.27)) (justify right))
+  )
+  (hierarchical_label "SWCLK" (shape output) (at 177.8 91.44 0) (fields_autoplaced)
+    (effects (font (size 1.27 1.27)) (justify left))
   )
   (hierarchical_label "IMP_LED" (shape input) (at 177.8 66.04 0) (fields_autoplaced)
@@
     (effects (font (size 1.27 1.27)) (justify right))
   )
+  (hierarchical_label "SWDIO" (shape output) (at 177.8 88.9 0) (fields_autoplaced)
+    (effects (font (size 1.27 1.27)) (justify left))
+  )
   (hierarchical_label "CAN1_RX" (shape input) (at 177.8 83.82 0) (fields_autoplaced)
