File: HARDWARE/TeR_ECU/TeR_ECU/TeR_ECU.kicad_sch (KiCad schematic)
At the start: 0 parts

Commit message: Menos el del conector grande, los demas esquematicos acabados
Other:
- removed sheet UniPort1
- removed sheet UniPort2
- added sheet Detección señales (Deteccion_señales.kicad_sch)
- added sheet Functions (Functions.kicad_sch)
- added sheet LV_BMS (UniPort.kicad_sch)
- added sheet LV_CAN (UniPort.kicad_sch)
- added sheet POWER (POWER.kicad_sch)
- added sheet PowerTrain (UniPort.kicad_sch)
- sheet CAN1: file CAN1.kicad_sch -> CAN.kicad_sch
- sheet CAN1 ports: added CAN+, CAN-, CAN_RX, CAN_TX; removed CAN1+, CAN1-, CAN1_RX, CAN1_TX
- sheet CAN2: file CAN2.kicad_sch -> CAN.kicad_sch
- sheet CAN2 ports: added CAN+, CAN-, CAN_RX, CAN_TX; removed CAN2+, CAN2-, CAN2_RX, CAN2_TX
- sheet Micro ports: added BL, BSPD_3V3, CAN1_RX, CAN1_TX, CAN2_RX, CAN2_TX, Horn, TSMS_3V3; removed none

Commit message: Listo para empezar con layout
Parts:
- added D3, D4, D5: LED, LED_SMD:LED_0805_2012Metric, symbol Device:LED
- added R18, R19, R20: 120R, Resistor_SMD:R_0805_2012Metric, symbol Device:R
Connections:
- new net: D5.2 (A), R20.2
- new net: D3.2 (A), R18.2
- new net: D4.2 (A), R19.2
- new net +3.3V: R20.1
- new net DBG_LED: R18.1
- new net GND: D3.1 (K), D4.1 (K), D5.1 (K)
- new net IMP_LED: R19.1
Other:
- added sheet Conector (Conector.kicad_sch)
- sheet Micro ports: added DBG_LED, IMP_LED; removed none
- note added: "Power"
- note added: "Status Leds"

Commit message: Revisar y empezar Layout
Other:
- sheet Conector ports: added LEDs; removed none
- sheet Micro ports: added LEDs; removed none
Changed lines of the file:
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@@
+    (stroke (width 0) (type default))
+  )
+  (wire (pts (xy 66.04 124.46) (xy 129.54 124.46))
     (stroke (width 0) (type default))
   )
@@
       (effects (font (size 1.27 1.27)) (justify left))
     )
+    (pin "LEDs" output (at 129.54 124.46 180)
+      (effects (font (size 1.27 1.27)) (justify left))
+    )
     (instances
       (project "TeR_ECU"
@@
       (effects (font (size 1.27 1.27)) (justify right))
     )
+    (pin "LEDs" input (at 66.04 124.46 0)
+      (effects (font (size 1.27 1.27)) (justify right))
+    )

Commit message: Revisar y empezar Layout
Other:
- sheet Conector ports: added SWCLK, SWDIO; removed none
- sheet Micro ports: added SWCLK, SWDIO; removed none
Changed lines of the file:
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@@
     (stroke (width 0) (type default))
   )
-  (wire (pts (xy 102.87 81.28) (xy 129.54 81.28))
+  (wire (pts (xy 109.22 81.28) (xy 129.54 81.28))
     (stroke (width 0) (type default))
   )
@@
     (stroke (width 0) (type default))
   )
-  (wire (pts (xy 102.87 105.41) (xy 129.54 105.41))
+  (wire (pts (xy 109.22 105.41) (xy 129.54 105.41))
     (stroke (width 0) (type default))
   )
@@
     (stroke (width 0) (type default))
   )
-  (wire (pts (xy 66.04 85.09) (xy 77.47 85.09))
+  (wire (pts (xy 66.04 85.09) (xy 83.82 85.09))
     (stroke (width 0) (type default))
   )
@@
     (stroke (width 0) (type default))
   )
-  (wire (pts (xy 102.87 85.09) (xy 129.54 85.09))
+  (wire (pts (xy 109.22 85.09) (xy 129.54 85.09))
     (stroke (width 0) (type default))
   )
@@
     (stroke (width 0) (type default))
   )
-  (wire (pts (xy 102.87 100.33) (xy 129.54 100.33))
+  (wire (pts (xy 109.22 100.33) (xy 129.54 100.33))
     (stroke (width 0) (type default))
   )
@@
     (stroke (width 0) (type default))
   )
-  (wire (pts (xy 66.04 81.28) (xy 77.47 81.28))
+  (wire (pts (xy 66.04 81.28) (xy 83.82 81.28))
+    (stroke (width 0) (type default))
+  )
+  (wire (pts (xy 66.04 121.92) (xy 129.54 121.92))
+    (stroke (width 0) (type default))
+  )
+  (wire (pts (xy 66.04 119.38) (xy 129.54 119.38))
     (stroke (width 0) (type default))
   )
@@
     (stroke (width 0) (type default))
   )
-  (wire (pts (xy 66.04 100.33) (xy 77.47 100.33))
+  (wire (pts (xy 66.04 100.33) (xy 83.82 100.33))
     (stroke (width 0) (type default))
   )
@@
     (stroke (width 0) (type default))
   )
-  (wire (pts (xy 66.04 105.41) (xy 77.47 105.41))
+  (wire (pts (xy 66.04 105.41) (xy 83.82 105.41))
     (stroke (width 0) (type default))
   )
@@
     )
   )
-  (sheet (at 77.47 95.25) (size 25.4 13.97) (fields_autoplaced)
-    (stroke (width 0.1524) (type solid))
-    (fill (color 0 0 0 0.0000))
-    (property "Sheetname" "Functions" (at 77.47 94.5384 0)
-      (effects (font (size 1.27 1.27)) (justify left bottom))
-    )
-    (property "Sheetfile" "Functions.kicad_sch" (at 77.47 109.8046 0)
-      (effects (font (size 1.27 1.27)) (justify left top))
-    )
-    (pin "Horn" input (at 102.87 105.41 0)
-      (effects (font (size 1.27 1.27)) (justify right))
-    )
-    (pin "BL" input (at 102.87 100.33 0)
-      (effects (font (size 1.27 1.27)) (justify right))
-    )
-    (pin "BL_GND" output (at 77.47 100.33 180)
-      (effects (font (size 1.27 1.27)) (justify left))
-    )
-    (pin "Horn_GND" output (at 77.47 105.41 180)
+  (sheet (at 83.82 95.25) (size 25.4 13.97) (fields_autoplaced)
+    (stroke (width 0.1524) (type solid))
+    (fill (color 0 0 0 0.0000))
+    (property "Sheetname" "Functions" (at 83.82 94.5384 0)
+      (effects (font (size 1.27 1.27)) (justify left bottom))
+    )
+    (property "Sheetfile" "Functions.kicad_sch" (at 83.82 109.8046 0)
+      (effects (font (size 1.27 1.27)) (justify left top))
+    )
+    (pin "Horn" input (at 109.22 105.41 0)
+      (effects (font (size 1.27 1.27)) (justify right))
+    )
+    (pin "BL" input (at 109.22 100.33 0)
+      (effects (font (size 1.27 1.27)) (justify right))
+    )
+    (pin "BL_GND" output (at 83.82 100.33 180)
+      (effects (font (size 1.27 1.27)) (justify left))
+    )
+    (pin "Horn_GND" output (at 83.82 105.41 180)
       (effects (font (size 1.27 1.27)) (justify left))
     )
@@
     )
   )
-  (sheet (at 77.47 77.47) (size 25.4 11.43) (fields_autoplaced)
-    (stroke (width 0.1524) (type solid))
-    (fill (color 0 0 0 0.0000))
-    (property "Sheetname" "Detección señales" (at 77.47 76.7584 0)
-      (effects (font (size 1.27 1.27)) (justify left bottom))
-    )
-    (property "Sheetfile" "Deteccion_señales.kicad_sch" (at 77.47 89.4846 0)
-      (effects (font (size 1.27 1.27)) (justify left top))
-    )
-    (pin "TSMS_3V3" output (at 102.87 85.09 0)
-      (effects (font (size 1.27 1.27)) (justify right))
-    )
-    (pin "TSMS_24V" input (at 77.47 85.09 180)
-      (effects (font (size 1.27 1.27)) (justify left))
-    )
-    (pin "BSPD_5V" input (at 77.47 81.28 180)
-      (effects (font (size 1.27 1.27)) (justify left))
-    )
-    (pin "BSPD_3V3" output (at 102.87 81.28 0)
+  (sheet (at 83.82 77.47) (size 25.4 11.43) (fields_autoplaced)
+    (stroke (width 0.1524) (type solid))
+    (fill (color 0 0 0 0.0000))
+    (property "Sheetname" "Detección señales" (at 83.82 76.7584 0)
+      (effects (font (size 1.27 1.27)) (justify left bottom))
+    )
+    (property "Sheetfile" "Deteccion_señales.kicad_sch" (at 83.82 89.4846 0)
+      (effects (font (size 1.27 1.27)) (justify left top))
+    )
+    (pin "TSMS_3V3" output (at 109.22 85.09 0)
+      (effects (font (size 1.27 1.27)) (justify right))
+    )
+    (pin "TSMS_24V" input (at 83.82 85.09 180)
+      (effects (font (size 1.27 1.27)) (justify left))
+    )
+    (pin "BSPD_5V" input (at 83.82 81.28 180)
+      (effects (font (size 1.27 1.27)) (justify left))
+    )
+    (pin "BSPD_3V3" output (at 109.22 81.28 0)
       (effects (font (size 1.27 1.27)) (justify right))
     )
@@
       (effects (font (size 1.27 1.27)) (justify left))
     )
+    (pin "SWCLK" output (at 129.54 121.92 180)
+      (effects (font (size 1.27 1.27)) (justify left))
+    )
+    (pin "SWDIO" output (at 129.54 119.38 180)
+      (effects (font (size 1.27 1.27)) (justify left))
+    )
     (instances
       (project "TeR_ECU"
@@
       (effects (font (size 1.27 1.27)) (justify right))
     )
+    (pin "SWCLK" input (at 66.04 121.92 0)
+      (effects (font (size 1.27 1.27)) (justify right))
+    )
+    (pin "SWDIO" input (at 66.04 119.38 0)
+      (effects (font (size 1.27 1.27)) (justify right))
+    )
