File: HARDWARE/TeR_ECU/TeR_ECU.kicad_pcb (KiCad board)
At the start: 4 copper layers, 105.4 x 62.7 mm, 68 parts, among them IC1 MX34040NF2, J1 Debug, J2 RJ45_Shielded, J3 RJ45_Shielded, J4 RJ45_Shielded, Q1 ZXMN3F30FH, Q2 ZXMN3F30FH, SW1 RST, U1 STM32F446RETx, U2 SN65HVD230, U3 SN65HVD230, U4 LM1117MP-3.3, U5 TSR_1-2450, U6 TSR_1-24120, U7 HDSP-A153, Y1 Crystal

Commit message: Rethought project using an STM32NucleoF7
Parts:
- removed C1: 10uF, Capacitor_SMD:C_0805_2012Metric
- removed C10, C13, C15: 100nF, Capacitor_SMD:C_0603_1608Metric
- removed C11, C12: 10pF, Capacitor_SMD:C_0603_1608Metric
- removed C14, C16: 4.7nF, Capacitor_SMD:C_0603_1608Metric
- removed C17, C18: 10u, Capacitor_SMD:C_0603_1608Metric
- removed C19, C20, C21, C22: 10 µF, Capacitor_SMD:C_0805_2012Metric
- removed C2, C3, C4, C5, C6: 100nF, Capacitor_SMD:C_0402_1005Metric
- removed C23: 4.7u, Capacitor_SMD:C_0805_2012Metric
- removed C7: 10nF, Capacitor_SMD:C_0402_1005Metric
- removed C8, C9: 1uF, Capacitor_SMD:C_0603_1608Metric
- removed D3: LED, LED_SMD:LED_0805_2012Metric
- removed D4, D5: NUP2105L, Package_TO_SOT_SMD:SOT-23
- removed F1: 500mA, Fuse:Fuse_0805_2012Metric
- removed FB1: 120R, Inductor_SMD:L_0805_2012Metric
- removed G***: LOGO, footprints:eracingLogo
- removed IC1: MX34040NF2, MX34040NF2:MX34040NF2
- removed J1: Debug, Connector_PinHeader_2.00mm:PinHeader_1x04_P2.00mm_Vertical
- removed J2, J3, J4: RJ45_Shielded, Connector_RJ:RJ45_Ninigi_GE
- removed JP1: BOOT0, Connector_PinHeader_2.00mm:PinHeader_1x03_P2.00mm_Vertical
- removed JP3, JP4: SolderJumper_3_Open, Jumper:SolderJumper-3_P1.3mm_Open_Pad1.0x1.5mm
- removed L1, L2: TCK-141, footprints:IND_TCK-141_TRP
- removed Q1, Q2: ZXMN3F30FH, Package_TO_SOT_SMD:SOT-23
- removed R1, R17, R20: 10k, Resistor_SMD:R_0805_2012Metric
- removed R10, R11, R8, R9: 50R, Resistor_SMD:R_0805_2012Metric
- removed R12: 25k5, Resistor_SMD:R_0805_2012Metric
- removed R13: 20k, Resistor_SMD:R_0805_2012Metric
- removed R14: 4k, Resistor_SMD:R_0805_2012Metric
- removed R15: 39k, Resistor_SMD:R_0805_2012Metric
- removed R16: 2k2, Resistor_SMD:R_0805_2012Metric
- removed R18, R19: 6R, Resistor_SMD:R_0805_2012Metric
- removed R3: 120R, Resistor_SMD:R_0805_2012Metric
- removed R4: 100R, Resistor_SMD:R_0603_1608Metric
- removed R5: 10k, Resistor_SMD:R_0603_1608Metric
- removed R7: 300R, Resistor_SMD:R_0402_1005Metric
- removed SW1: RST, Button_Switch_SMD:SW_Tactile_SPST_NO_Straight_CK_PTS636Sx25SMTRLFS
- removed U1: STM32F446RETx, Package_QFP:LQFP-64_10x10mm_P0.5mm
- removed U2, U3: SN65HVD230, Package_SO:SOIC-8_3.9x4.9mm_P1.27mm
- removed U4: LM1117MP-3.3, Package_TO_SOT_SMD:SOT-223-3_TabPin2
- removed U5: TSR_1-2450, Converter_DCDC:Converter_DCDC_TRACO_TSR-1_THT
- removed U6: TSR_1-24120, Converter_DCDC:Converter_DCDC_TRACO_TSR-1_THT
- removed U7: HDSP-A153, Display_7Segment:HDSP-A151
- removed Y1: Crystal, Crystal:Crystal_SMD_5032-2Pin_5.0x3.2mm
Routing:
- net +24V: track 132.3 -> 0.00 mm, vias 2 -> 0
- net +12V: track 94.2 -> 0.00 mm
- net +5V: track 89.0 -> 0.00 mm, vias 1 -> 0
- net GND: track 68.1 -> 0.00 mm, vias 30 -> 0
- net /Micro/SWCLK: track 48.9 -> 0.00 mm, vias 1 -> 0
- net /Micro/SWDIO: track 46.4 -> 0.00 mm, vias 1 -> 0
- net /24V_IN: track 46.2 -> 0.00 mm, vias 1 -> 0
- net +3.3V: track 41.9 -> 0.00 mm, vias 14 -> 0
- net /CAN_MAIN/CAN-: track 41.8 -> 0.00 mm
- net /Conector/UART_RX: track 41.1 -> 0.00 mm
- net /Conector/UART_TX: track 41.1 -> 0.00 mm
- net /CAN_MAIN/CAN+: track 41.0 -> 0.00 mm
- net /Conector/LEDs: track 38.7 -> 0.00 mm
- net /Functions/Horn: track 35.5 -> 0.00 mm
- net /Functions/BL: track 26.9 -> 0.00 mm
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- removed copper zone on In2.Cu, net +3.3V
- removed copper zone on In2.Cu, net /24V_IN
- removed copper zone on In1.Cu, net GND
Other:
- board outline removed
- board text removed: "0"
- board text removed: "1"
- board text removed: "BOOT0"
- board text removed: "DEBUG"
- board text removed: "PWR"
- board text removed: "Reset"
- board text removed: "Status"
- board text removed: "TeR_ECU V1.0.0 Idiazriofri Ozuba 2023"

Commit message: Replanteado layout con una F7
Parts:
- added C13: 100nF, Capacitor_SMD:C_0603_1608Metric, F.Cu at (131.0, 67.0)
- added C14: 4.7nF, Capacitor_SMD:C_0603_1608Metric, F.Cu at (133.5, 67.0)
- added C15: 100nF, Capacitor_SMD:C_0603_1608Metric, F.Cu at (131.0, 83.1)
- added C16: 4.7nF, Capacitor_SMD:C_0603_1608Metric, F.Cu at (133.5, 83.1)
- added C17: 10u, Capacitor_SMD:C_0603_1608Metric, F.Cu at (117.2, 75.7)
- added C18: 10u, Capacitor_SMD:C_0603_1608Metric, F.Cu at (119.7, 75.7)
- added C19: 10 µF, Capacitor_SMD:C_0805_2012Metric, F.Cu at (102.1, 71.9)
- added C20: 10 µF, Capacitor_SMD:C_0805_2012Metric, F.Cu at (105.1, 71.9)
- added D3: LED, LED_SMD:LED_0805_2012Metric, F.Cu at (124.8, 98.6)
- added D4: NUP2105L, Package_TO_SOT_SMD:SOT-23, F.Cu at (131.9, 75.9)
- added D5: NUP2105L, Package_TO_SOT_SMD:SOT-23, F.Cu at (131.9, 92.0)
- added F1: 500mA, Fuse:Fuse_0805_2012Metric, F.Cu at (108.1, 71.9)
- added IC1: MX34040NF2, MX34040NF2:MX34040NF2, F.Cu at (181.5, 132.1)
- added J2: RJ45_Shielded, Connector_RJ:RJ45_Ninigi_GE, F.Cu at (101.3, 131.5)
- added J3: RJ45_Shielded, Connector_RJ:RJ45_Ninigi_GE, F.Cu at (123.6, 131.5)
- added J4: RJ45_Shielded, Connector_RJ:RJ45_Ninigi_GE, F.Cu at (79.0, 131.5)
- added JP3: SolderJumper_3_Open, Jumper:SolderJumper-3_P1.3mm_Open_Pad1.0x1.5mm, F.Cu at (125.0, 67.0)
- added JP4: SolderJumper_3_Open, Jumper:SolderJumper-3_P1.3mm_Open_Pad1.0x1.5mm, F.Cu at (125.0, 83.1)
- added L1: TCK-141, footprints:IND_TCK-141_TRP, F.Cu at (112.9, 73.9)
- added Q1: ZXMN3F30FH, Package_TO_SOT_SMD:SOT-23, F.Cu at (102.8, 60.8)
- added Q2: ZXMN3F30FH, Package_TO_SOT_SMD:SOT-23, F.Cu at (107.2, 60.8)
- added R1: 10k, Resistor_SMD:R_0805_2012Metric, F.Cu at (102.0, 65.4)
- added R10: 50R, Resistor_SMD:R_0805_2012Metric, F.Cu at (131.2, 87.3)
- added R11: 50R, Resistor_SMD:R_0805_2012Metric, F.Cu at (134.2, 87.3)
- added R12: 25k5, Resistor_SMD:R_0805_2012Metric, F.Cu at (124.8, 60.0)
- added R13: 20k, Resistor_SMD:R_0805_2012Metric, F.Cu at (127.7, 60.0)
- added R14: 4k, Resistor_SMD:R_0805_2012Metric, F.Cu at (130.7, 60.0)
- added R15: 39k, Resistor_SMD:R_0805_2012Metric, F.Cu at (133.6, 60.0)
- added R16: 2k2, Resistor_SMD:R_0805_2012Metric, F.Cu at (105.0, 65.4)
- added R17: 10k, Resistor_SMD:R_0805_2012Metric, F.Cu at (108.0, 65.4)
- added R18: 6R, Resistor_SMD:R_0805_2012Metric, F.Cu at (110.9, 65.4)
- added R19: 6R, Resistor_SMD:R_0805_2012Metric, F.Cu at (113.8, 65.4)
- added R20: 10k, Resistor_SMD:R_0805_2012Metric, F.Cu at (116.8, 65.4)
- added R3: 120R, Resistor_SMD:R_0805_2012Metric, F.Cu at (127.8, 98.6)
- added R8: 50R, Resistor_SMD:R_0805_2012Metric, F.Cu at (131.2, 71.2)
- added R9: 50R, Resistor_SMD:R_0805_2012Metric, F.Cu at (134.2, 71.2)
- added U2: SN65HVD230, Package_SO:SOIC-8_3.9x4.9mm_P1.27mm, F.Cu at (126.5, 74.1)
- added U3: SN65HVD230, Package_SO:SOIC-8_3.9x4.9mm_P1.27mm, F.Cu at (126.5, 90.2)
- added U4: LM1117MP-3.3, Package_TO_SOT_SMD:SOT-223-3_TabPin2, F.Cu at (114.1, 82.6)
- added U5: TSR_1-2450, Converter_DCDC:Converter_DCDC_TRACO_TSR-1_THT, F.Cu at (107.0, 83.2)
- added U7: HDSP-A153, Display_7Segment:HDSP-A151, F.Cu at (149.8, 143.0)
- added U8: NUCLEO144-F746ZG, Module:ST_Morpho_Connector_144_STLink, F.Cu at (175.4, 44.8)

Commit message: Empezando Layout
Parts:
- removed U8: NUCLEO144-F746ZG, Module:ST_Morpho_Connector_144_STLink
- added U1: NUCLEO-F446RE, Nucleo-F446RE:MODULE_NUCLEO-F446RE, F.Cu at (111.3, 79.0)
- moved J4 82.8 mm to (60.6, 50.8), turned to -90 degrees
- moved J3 72.6 mm to (60.6, 95.4), turned to -90 degrees
- moved J2 71.2 mm to (60.6, 73.1), turned to -90 degrees
- moved U5 61.7 mm to (158.9, 49.9), turned to 0 degrees
- moved D4 58.9 mm to (76.4, 95.6), turned to 180 degrees
- moved R9 57.5 mm to (80.9, 93.1), turned to 180 degrees
- moved R8 56.6 mm to (81.3, 97.9), turned to 0 degrees
- moved IC1 56.4 mm to (184.4, 75.7), turned to 90 degrees
- moved D5 53.9 mm to (78.7, 83.9), turned to 180 degrees
- moved R11 51.8 mm to (82.7, 81.4), turned to 180 degrees
- moved C14 51.0 mm to (88.8, 91.6), turned to 0 degrees
- moved JP3 49.2 mm to (85.0, 95.6)
- moved R10 48.5 mm to (82.7, 86.2), turned to 0 degrees
- moved C13 45.3 mm to (95.9, 95.6)
- moved C16 44.5 mm to (89.0, 80.4), turned to 180 degrees
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Routing:
- net /CAN_POWERTRAIN/CAN-: track 0.00 -> 57.3 mm
- net /CAN_POWERTRAIN/CAN+: track 0.00 -> 54.4 mm
- net /CAN_MAIN/CAN-: track 0.00 -> 54.3 mm
- net /CAN_MAIN/CAN+: track 0.00 -> 52.8 mm
- net GND: track 0.00 -> 31.2 mm, vias 0 -> 6
- net /CAN_MAIN/CAN_RX: track 0.00 -> 20.7 mm, vias 0 -> 1
- net /CAN_POWERTRAIN/VREF: track 0.00 -> 14.7 mm, vias 0 -> 2
- net /CAN_MAIN/CAN_TX: track 0.00 -> 14.1 mm
- net /CAN_MAIN/VREF: track 0.00 -> 13.0 mm, vias 0 -> 2
- net +3.3V: track 0.00 -> 5.83 mm
- net Net-(JP3-B): track 0.00 -> 3.67 mm
- net Net-(JP4-B): track 0.00 -> 3.16 mm
- net Net-(JP3-A): track 0.00 -> 3.16 mm
- net Net-(JP4-A): track 0.00 -> 3.05 mm
- added copper zone on In1.Cu, net GND

Commit message: Layout acabado
Parts:
- moved C20 68.8 mm to (160.3, 110.9)
- moved C19 67.5 mm to (147.7, 112.1), turned to -90 degrees
- moved F1 65.3 mm to (142.0, 111.2), turned to 0 degrees
- moved L1 63.9 mm to (154.4, 111.2), turned to 180 degrees
- moved C17 56.4 mm to (168.2, 103.0)
- moved U5 55.4 mm to (157.4, 105.3)
- moved C18 49.9 mm to (148.7, 99.6), turned to 0 degrees
- moved U4 37.3 mm to (151.5, 93.7), turned to 180 degrees
- moved R16 21.7 mm to (126.3, 61.2), turned to 0 degrees
- moved R19 17.4 mm to (97.5, 59.3), turned to 180 degrees
- moved Q1 15.5 mm to (118.3, 61.2), turned to 0 degrees
- moved R3 15.4 mm to (162.7, 82.5), turned to -90 degrees
- moved R17 14.7 mm to (122.3, 62.1), turned to -90 degrees
- moved D3 12.1 mm to (162.7, 86.2)
- moved U7 11.2 mm to (172.2, 111.7)
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Connections:
- U1 pad CN10_27: /Detección señales/TSMS_3V3 -> unconnected-(U1B-PB4-PadCN10_27)
- U1 pad CN10_31: /Detección señales/BSPD_3V3 -> unconnected-(U1B-PB3-PadCN10_31)
- U1 pad CN7_30: unconnected-(U1A-PA1-PadCN7_30) -> /Functions/Horn
- U1 pad CN7_32: unconnected-(U1A-PA4-PadCN7_32) -> /Detección señales/TSMS_3V3
- U1 pad CN7_34: /Functions/Horn -> /Detección señales/BSPD_3V3
Routing:
- net +5V: track 0.00 -> 109.7 mm, vias 0 -> 2
- net +24V: track 0.00 -> 104.0 mm, vias 0 -> 3
- net +3.3V: track 5.83 -> 105.8 mm, vias 0 -> 5
- net /Conector/BSPD_5V: track 0.00 -> 92.0 mm
- net /Conector/TSMS_24V: track 0.00 -> 85.6 mm
- net /Conector/Horn_GND: track 0.00 -> 70.4 mm
- net /Conector/UART_TX: track 0.00 -> 59.0 mm
- net /Conector/UART_RX: track 0.00 -> 58.8 mm
- net /24V_IN: track 0.00 -> 55.6 mm, vias 0 -> 1
- net /Conector/BL_GND: track 0.00 -> 46.6 mm
- net /CAN_POWERTRAIN/CAN_RX: track 0.00 -> 39.6 mm
- net /CAN_POWERTRAIN/CAN_TX: track 0.00 -> 32.0 mm
- net /Functions/BL: track 0.00 -> 26.8 mm, vias 0 -> 1
- net GND: track 31.2 -> 56.0 mm, vias 6 -> 18
- net /Functions/Horn: track 0.00 -> 17.5 mm
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- added copper zone on In2.Cu, net +3.3V
- added copper zone on In2.Cu, net +5V
- added copper zone on In2.Cu, net /24V_IN

Commit message: Layout acabado
Parts:
- moved U7 67.7 mm to (151.0, 47.4)
- moved R13 46.6 mm to (127.7, 48.0), turned to -90 degrees
- moved R15 42.9 mm to (124.8, 47.9), turned to 90 degrees
- moved R14 38.9 mm to (127.7, 54.0), turned to 90 degrees
- moved R12 36.4 mm to (124.7, 54.0), turned to -90 degrees
- moved C17 35.7 mm to (132.5, 101.6), turned to 0 degrees
- moved U4 34.5 mm to (119.3, 106.3)
- moved C18 34.5 mm to (116.5, 112.2)
- moved R3 32.0 mm to (150.5, 112.1)
- moved D3 32.0 mm to (150.6, 115.8)
- moved C20 27.9 mm to (132.7, 115.3)
- moved F1 27.9 mm to (114.4, 115.7)
- moved U5 27.9 mm to (129.8, 109.7)
- moved C19 27.9 mm to (120.1, 116.5)
- moved L1 27.9 mm to (126.8, 115.6)
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Connections:
- U1 pad CN7_21: /Functions/BL -> /Functions/Horn
- U1 pad CN7_30: /Functions/Horn -> /Functions/BL
Routing:
- net +5V: track 109.7 -> 46.8 mm
- net /CAN_MAIN/CAN_RX: track 20.7 -> 70.6 mm
- net /CAN_MAIN/CAN_TX: track 14.1 -> 59.5 mm
- net /Conector/BSPD_5V: track 92.0 -> 47.4 mm
- net /Conector/UART_TX: track 59.0 -> 25.4 mm
- net /Conector/UART_RX: track 58.8 -> 26.7 mm
- net /Conector/TSMS_24V: track 85.6 -> 58.8 mm
- net /24V_IN: track 55.6 -> 30.3 mm, vias 1 -> 2
- net /CAN_POWERTRAIN/CAN_RX: track 39.6 -> 15.4 mm
- net /Functions/Horn: track 17.5 -> 34.5 mm
- net +24V: track 104.0 -> 119.1 mm
- net /CAN_POWERTRAIN/CAN+: track 54.4 -> 69.2 mm
- net /CAN_POWERTRAIN/CAN-: track 57.3 -> 68.9 mm
- net /Conector/Horn_GND: track 70.4 -> 61.2 mm
- net /Functions/BL: track 26.8 -> 21.1 mm, vias 1 -> 0
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
Commit message: revisar
Parts:
- moved U7 2.44 mm to (149.7, 49.5)
Routing:
- net /CAN_POWERTRAIN/CAN+: track 69.2 -> 66.9 mm
- net /CAN_POWERTRAIN/CAN-: track 68.9 -> 68.3 mm
Other:
- board outline added: 115.3 x 84.8 mm
Changed lines of the file:
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@@
   )
   (footprint "Display_7Segment:HDSP-A151" (layer "F.Cu")
-    (at 150.9525 47.3775 90)
+    (at 149.6685 49.4575 90)
     (descr "One digit 7 segment red, https://docs.broadcom.com/docs/AV02-2553EN")
     (tags "One digit 7 segment high efficiency red")
@@
     )
   )
+  (gr_line (start 158.496 122.682) (end 164.084 117.094)
+    (stroke (width 0.1) (type default)) (layer "Edge.Cuts"))
+  (gr_line (start 164.084 117.094) (end 164.084 43.434)
+    (stroke (width 0.1) (type default)) (layer "Edge.Cuts"))
+  (gr_line (start 48.768 43.434) (end 54.356 37.846)
+    (stroke (width 0.1) (type default)) (layer "Edge.Cuts"))
+  (gr_line (start 48.768 43.434) (end 48.768 117.094)
+    (stroke (width 0.1) (type default)) (layer "Edge.Cuts"))
+  (gr_line (start 158.496 37.846) (end 164.084 43.434)
+    (stroke (width 0.1) (type default)) (layer "Edge.Cuts"))
+  (gr_line (start 54.356 122.682) (end 158.496 122.682)
+    (stroke (width 0.1) (type default)) (layer "Edge.Cuts"))
+  (gr_line (start 48.768 117.094) (end 54.356 122.682)
+    (stroke (width 0.1) (type default)) (layer "Edge.Cuts"))
+  (gr_line (start 158.496 37.846) (end 54.356 37.846)
+    (stroke (width 0.1) (type default)) (layer "Edge.Cuts"))
   (segment (start 124.825 45.005) (end 124.825 44.995) (width 0.25) (layer "F.Cu") (net 1))
   (segment (start 91.059 108.85) (end 92.539 108.85) (width 0.2) (layer "F.Cu") (net 1))
@@
   (segment (start 62.14 74.61) (end 60.65 73.12) (width 0.2) (layer "B.Cu") (net 10))
   (segment (start 60.65 95.395) (end 62.739999 93.305001) (width 0.2) (layer "B.Cu") (net 10))
-  (segment (start 73.535 94.906104) (end 73.535 63.093603) (width 0.2) (layer "F.Cu") (net 11))
   (segment (start 75.2205 100.891) (end 75.2205 100.9945) (width 0.2) (layer "F.Cu") (net 11))
+  (segment (start 82.968604 99.24) (end 83.31 99.24) (width 0.2) (layer "F.Cu") (net 11))
+  (segment (start 70.866 97.575104) (end 70.866 60.424603) (width 0.2) (layer "F.Cu") (net 11))
+  (segment (start 73.085 99.555) (end 73.527 99.555) (width 0.2) (layer "F.Cu") (net 11))
   (segment (start 73.535 99.105) (end 73.535 99.005) (width 0.2) (layer "F.Cu") (net 11))
-  (segment (start 82.968604 99.24) (end 83.31 99.24) (width 0.2) (layer "F.Cu") (net 11))
+  (segment (start 80.301604 101.907) (end 82.968604 99.24) (width 0.2) (layer "F.Cu") (net 11))
+  (segment (start 73.085 99.555) (end 73.535 99.105) (width 0.2) (layer "F.Cu") (net 11))
+  (segment (start 70.1725 98.941396) (end 70.1725 98.268604) (width 0.2) (layer "F.Cu") (net 11))
+  (segment (start 70.436104 99.205) (end 70.1725 98.941396) (width 0.2) (layer "F.Cu") (net 11))
+  (segment (start 63.19 52.748603) (end 63.19 52.115) (width 0.2) (layer "F.Cu") (net 11))
+  (segment (start 74.863 100.891) (end 75.2205 100.891) (width 0.2) (layer "F.Cu") (net 11))
   (segment (start 73.535 99.005) (end 72.183896 99.005) (width 0.2) (layer "F.Cu") (net 11))
-  (segment (start 73.535 63.093603) (end 63.19 52.748603) (width 0.2) (layer "F.Cu") (net 11))
-  (segment (start 73.085 99.555) (end 73.535 99.105) (width 0.2) (layer "F.Cu") (net 11))
-  (segment (start 63.19 52.748603) (end 63.19 52.115) (width 0.2) (layer "F.Cu") (net 11))
   (segment (start 72.183896 99.005) (end 71.983896 99.205) (width 0.2) (layer "F.Cu") (net 11))
-  (segment (start 73.085 99.555) (end 73.527 99.555) (width 0.2) (layer "F.Cu") (net 11))
-  (segment (start 80.301604 101.907) (end 82.968604 99.24) (width 0.2) (layer "F.Cu") (net 11))
-  (segment (start 70.436104 99.205) (end 70.1725 98.941396) (width 0.2) (layer "F.Cu") (net 11))
-  (segment (start 70.1725 98.268604) (end 73.535 94.906104) (width 0.2) (layer "F.Cu") (net 11))
-  (segment (start 74.863 100.891) (end 75.2205 100.891) (width 0.2) (layer "F.Cu") (net 11))
-  (segment (start 70.1725 98.941396) (end 70.1725 98.268604) (width 0.2) (layer "F.Cu") (net 11))
+  (segment (start 75.2205 100.9945) (end 76.133 101.907) (width 0.2) (layer "F.Cu") (net 11))
   (segment (start 71.983896 99.205) (end 70.436104 99.205) (width 0.2) (layer "F.Cu") (net 11))
-  (segment (start 75.2205 100.9945) (end 76.133 101.907) (width 0.2) (layer "F.Cu") (net 11))
+  (segment (start 70.866 60.424603) (end 63.19 52.748603) (width 0.2) (layer "F.Cu") (net 11))
   (segment (start 73.527 99.555) (end 74.863 100.891) (width 0.2) (layer "F.Cu") (net 11))
+  (segment (start 70.1725 98.268604) (end 70.866 97.575104) (width 0.2) (layer "F.Cu") (net 11))
   (segment (start 76.133 101.907) (end 80.301604 101.907) (width 0.2) (layer "F.Cu") (net 11))
-  (segment (start 62.755075 51.065) (end 62.14 51.680075) (width 0.2) (layer "F.Cu") (net 12))
+  (segment (start 64.24 53.232917) (end 64.24 51.680075) (width 0.2) (layer "F.Cu") (net 12))
   (segment (start 73.56 97.655) (end 73.085 97.655) (width 0.2) (layer "F.Cu") (net 12))
+  (segment (start 62.14 51.680075) (end 62.14 52.335) (width 0.2) (layer "F.Cu") (net 12))
   (segment (start 75.15 96.065) (end 73.56 97.655) (width 0.2) (layer "F.Cu") (net 12))
   (segment (start 76.2365 95.049) (end 79.943 95.049) (width 0.2) (layer "F.Cu") (net 12))
+  (segment (start 62.755075 51.065) (end 62.14 51.680075) (width 0.2) (layer "F.Cu") (net 12))
+  (segment (start 71.747 97.655) (end 71.266 97.174) (width 0.2) (layer "F.Cu") (net 12))
+  (segment (start 71.266 60.258918) (end 64.24 53.232917) (width 0.2) (layer "F.Cu") (net 12))
+  (segment (start 71.266 97.174) (end 71.266 60.258918) (width 0.2) (layer "F.Cu") (net 12))
   (segment (start 75.2205 96.065) (end 75.15 96.065) (width 0.2) (layer "F.Cu") (net 12))
+  (segment (start 62.14 52.335) (end 60.65 50.845) (width 0.2) (layer "F.Cu") (net 12))
   (segment (start 79.943 95.049) (end 82.864 97.97) (width 0.2) (layer "F.Cu") (net 12))
   (segment (start 64.24 51.680075) (end 63.624925 51.065) (width 0.2) (layer "F.Cu") (net 12))
-  (segment (start 64.24 52.549925) (end 64.24 51.680075) (width 0.2) (layer "F.Cu") (net 12))
-  (segment (start 62.14 51.680075) (end 62.14 52.335) (width 0.2) (layer "F.Cu") (net 12))
-  (segment (start 73.085 97.50498) (end 73.721388 97.50498) (width 0.2) (layer "F.Cu") (net 12))
   (segment (start 82.864 97.97) (end 83.31 97.97) (width 0.2) (layer "F.Cu") (net 12))
-  (segment (start 73.98498 97.241388) (end 73.98498 62.907215) (width 0.2) (layer "F.Cu") (net 12))
-  (segment (start 73.085 97.655) (end 73.085 97.50498) (width 0.2) (layer "F.Cu") (net 12))
+  (segment (start 63.624925 51.065) (end 62.755075 51.065) (width 0.2) (layer "F.Cu") (net 12))
+  (segment (start 73.085 97.655) (end 71.747 97.655) (width 0.2) (layer "F.Cu") (net 12))
   (segment (start 75.2205 96.065) (end 76.2365 95.049) (width 0.2) (layer "F.Cu") (net 12))
-  (segment (start 62.14 52.335) (end 60.65 50.845) (width 0.2) (layer "F.Cu") (net 12))
-  (segment (start 73.98498 62.907215) (end 63.933845 52.85608) (width 0.2) (layer "F.Cu") (net 12))
-  (segment (start 63.624925 51.065) (end 62.755075 51.065) (width 0.2) (layer "F.Cu") (net 12))
-  (segment (start 73.721388 97.50498) (end 73.98498 97.241388) (width 0.2) (layer "F.Cu") (net 12))
-  (segment (start 63.933845 52.85608) (end 64.24 52.549925) (width 0.2) (layer "F.Cu") (net 12))
   (segment (start 153.96 98.19) (end 153.96 95.99) (width 0.35) (layer "F.Cu") (net 13))
   (segment (start 110.82895 115.65) (end 110.72895 115.65) (width 0.25) (layer "F.Cu") (net 13))
