File: HARDWARE/TeR_ECU/IMU.kicad_sch (KiCad schematic)
At the start: 6 parts, among them U6 ASM330LHH

Commit message: Cool things
Parts:
- removed R29, R30: 10k, symbol Device:R_Small
- added U9: LIS3MDL, Package_LGA:LGA-12_2x2mm_P0.5mm, symbol Sensor_Magnetic:LIS3MDL
Connections:
- net GND: now also U9.12 (GND), U9.2 (GND), U9.3 (GND)
- net SCL: now also U9.1 (SCL/SPC)
- net SDA: now also U9.11 (SDA/SDI/SDO)
- no-connect marks 7 -> 9
Other:
- moved on the sheet: C30, C31, C32, U6

Commit message: Quick changes, go to start layouting
Parts:
- added C35, C37: 100n, Capacitor_SMD:C_0603_1608Metric, symbol Device:C_Small
- added C36: 1u, Capacitor_SMD:C_0603_1608Metric, symbol Device:C_Small
- C34: renamed from C30; footprint (none) -> Capacitor_SMD:C_0603_1608Metric
- C38: renamed from C31; footprint (none) -> Capacitor_SMD:C_0603_1608Metric
- C39: renamed from C32; footprint (none) -> Capacitor_SMD:C_0603_1608Metric
- renumbered U6 to U8
Connections:
- net +3.3V: now also U9.5 (Vdd), U9.6 (Vdd_IO), C36.2, C37.2
- net GND: now also U9.9 (SDO/SA1), C35.2, C36.1, C37.1
- net at U9.4 (C1): now also C35.1
- no-connect marks 9 -> 11
Other:
- moved on the sheet: U9

Commit message: Began layout
Parts:
- U8: footprint LGA-14L_2P5X3X0P83_STM -> IMU:LGA-14L_2P5X3X0P83_STM-L
Changed lines of the file:
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@@
 			)
 		)
-		(property "Footprint" "LGA-14L_2P5X3X0P83_STM"
+		(property "Footprint" "IMU:LGA-14L_2P5X3X0P83_STM-L"
 			(at 128.27 125.73 0)
 			(effects

Commit message: Finished layout, RF design, and quick DRC check, Lookin gud
Connections:
- net +3.3V: now also U8.12 (CS), U8.2 (RES), U8.3 (RES), U9.10 (~{CS})
- net GND: now also U8.1 (SDO/SA0)
- no-connect marks 11 -> 6
Other:
- note added: "Accel + Gyro"
- note added: "Address 0b0011100"
- note added: "Address 0b1101010"
- note added: "Magnetometer"
- moved on the sheet: C36
