File: HARDWARE/TeR_ECU/IMU.kicad_sch (KiCad schematic)
At the start: 8 parts, among them U8 ASM330LHH, U9 LIS3MDL

Commit message: Corregidos conectores, CAN y añadidas librerias al proyecto para cargar huellas
Parts:
- U8: footprint IMU:LGA-14L_2P5X3X0P83_STM-L -> ASM330:LGA-14L_2P5X3X0P83_STM-L
