File: HARDWARE/TeR_ECU/INPUTS.kicad_sch (KiCad schematic)
At the start: 8 parts

Commit message: Cool things
Parts:
- added C36, C37, C38, C39: 20n, symbol Device:C_Small
- added D11, D12, D13, D14, D15, D16, D17, D18: SMAJ26A, Diode_SMD:D_SMA, symbol Diode:SMAJ26A
- added R37, R40, R42, R44: 10k, symbol Device:R_Small
- added R38, R39, R41, R43: 0R, symbol Device:R_Small
- added R45, R46, R47, R48: 1K, symbol Device:R_Small
- added U10: LM324, symbol Amplifier_Operational:LM324
Connections:
- net D4 is gone; now on net D3: D9.1 (K), R9.2
- net D1: now also D7.1 (K), R7.2; no longer D10.1 (K), R10.2
- net D2: now also D8.1 (K), R8.2; no longer D7.1 (K), R7.2
- net D3: no longer D8.1 (K), R8.2
- net DIN0: now also D11.2 (A2); no longer R8.1, R9.1
- net DIN1: now also D12.2 (A2)
- net GND: now also C36.2, C37.2, C38.2, C39.2, D11.1 (A1), D12.1 (A1), D13.1 (A1), D14.1 (A1), D15.1 (A1), D16.1 (A1), D17.1 (A1), D18.1 (A1), R37.2, R40.2, R42.2, R44.2, U10.11 (V-)
- new net: R37.1, R38.2, U10.3 (+)
- new net: R43.2, R44.1, U10.12 (+)
- new net: R39.2, R40.1, U10.5 (+)
- new net: R46.1, U10.6 (-), U10.7
- new net: R45.1, U10.1, U10.2 (-)
- new net: R48.1, U10.13 (-), U10.14
- new net: R41.2, R42.1, U10.10 (+)
- new net: R47.1, U10.8, U10.9 (-)
- new net +3.3V: U10.4 (V+)
- new net A0: C36.1, R45.2
- new net A1: C37.1, R46.2
- new net A2: C38.1, R47.2
- new net A3: C39.1, R48.2
- new net AIN0: D16.2 (A2), R38.1
- new net AIN1: D15.2 (A2), R39.1
- new net AIN2: D17.2 (A2), R41.1
- new net AIN3: D18.2 (A2), R43.1
- new net D0: D10.1 (K), R10.2
- new net DIN2: D13.2 (A2), R8.1
- new net DIN3: D14.2 (A2), R9.1
Other:
- note added: "ANALOG INPUTS"
- note added: "Filters Calculated for a 5khz lowpass antialias, antinoise filter, mainly for reading sensors at human freq."
- note added: "With This circuit you can ensure operation at a whole range of input voltage, zener current clamps to archieve desired voltage."
- moved on the sheet: D10, D7, D8, D9, R10, R7, R8, R9

Commit message: Quick changes, go to start layouting
Parts:
- C13: renamed from C36; footprint (none) -> Capacitor_SMD:C_0603_1608Metric
- C14: renamed from C37; footprint (none) -> Capacitor_SMD:C_0603_1608Metric
- C15: renamed from C38; footprint (none) -> Capacitor_SMD:C_0603_1608Metric
- C16: renamed from C39; footprint (none) -> Capacitor_SMD:C_0603_1608Metric
- renumbered D12 to D11, D7 to D12, D8 to D14, D14 to D15, D9 to D16, D16 to D17, D15 to D18, D17 to D19, D18 to D20, D11 to D9, R10 to R11, R7 to R12, R8 to R13, R9 to R14, R38 to R15, R39 to R16, R41 to R17, R43 to R18, R37 to R19, R40 to R20, R42 to R21, R44 to R22, R45 to R23, R46 to R24, R47 to R25, R48 to R26, U10 to U5

Commit message: Began layout
Parts:
- removed D11, D13, D15, D17, D18, D19, D20, D9: SMAJ26A, Diode_SMD:D_SMA, symbol Diode:SMAJ26A
- added D11, D13, D15, D17, D18, D19, D20, D9: PTVS26VZ1USK, Diode_SMD:Nexperia_DSN1608-2_1.6x0.8mm, symbol Diode:PTVS26VZ1USK
- R15, R16, R17, R18, R19, R20, R21, R22, R23, R24, R25, R26: footprint (none) -> Resistor_SMD:R_0603_1608Metric
- U5: footprint (none) -> Package_SO:SOIC-14_3.9x8.7mm_P1.27mm
Connections:
- net AIN0: now also D17.2 (A)
- net AIN1: now also D18.2 (A)
- net AIN2: now also D19.2 (A)
- net AIN3: now also D20.2 (A)
- net DIN0: now also D9.2 (A)
- net DIN1: now also D11.2 (A)
- net DIN2: now also D13.2 (A)
- net DIN3: now also D15.2 (A)
- net GND: now also D11.1 (K), D13.1 (K), D15.1 (K), D17.1 (K), D18.1 (K), D19.1 (K), D20.1 (K), D9.1 (K)
Other:
- moved on the sheet: D12, D14, D16, R12, R13, R14, U5E

Commit message: First layout prototype
Parts:
- removed D10, D12, D14, D16: BZV55B3V3, Diode_SMD:D_MiniMELF, symbol Diode:BZV55B3V3
- added D10, D12, D14, D31: SZMM5Z3V3T1G, Diode_SMD:D_SOD-523, symbol Device:D_Zener
- R11, R12, R13, R14: footprint Resistor_SMD:R_0805_2012Metric -> Resistor_SMD:R_0603_1608Metric
Connections:
- net D0: now also D14.1 (K)
- net D1: now also D12.1 (K)
- net D2: now also D10.1 (K)
- net D3: now also D31.1 (K)
- net GND: now also D10.2 (A), D12.2 (A), D14.2 (A), D31.2 (A)

Commit message: Finished layout, RF design, and quick DRC check, Lookin gud
Connections:
- net AIN0: now also D17.1 (K); no longer D17.2 (A)
- net AIN1: now also D18.1 (K); no longer D18.2 (A)
- net AIN2: now also D19.1 (K); no longer D19.2 (A)
- net AIN3: now also D20.1 (K); no longer D20.2 (A)
- net DIN0: now also D9.1 (K); no longer D9.2 (A)
- net DIN1: now also D11.1 (K); no longer D11.2 (A)
- net DIN2: now also D13.1 (K); no longer D13.2 (A)
- net DIN3: now also D15.1 (K); no longer D15.2 (A)
- net GND: now also D11.2 (A), D13.2 (A), D15.2 (A), D17.2 (A), D18.2 (A), D19.2 (A), D20.2 (A), D9.2 (A); no longer D11.1 (K), D13.1 (K), D15.1 (K), D17.1 (K), D18.1 (K), D19.1 (K), D20.1 (K), D9.1 (K)
Changed lines of the file:
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@@
 		(lib_id "Diode:PTVS26VZ1USK")
 		(at 173.99 105.41 270)
-		(mirror x)
 		(unit 1)
 		(exclude_from_sim no)
@@
 		(dnp no)
 		(property "Reference" "D19"
-			(at 171.45 104.1399 90)
+			(at 171.45 106.6801 90)
 			(effects
 				(font
@@
 		)
 		(property "Value" "PTVS26VZ1USK"
-			(at 171.45 106.6799 90)
+			(at 171.45 104.1401 90)
 			(effects
 				(font
@@
 		(lib_id "Diode:PTVS26VZ1USK")
 		(at 173.99 129.54 270)
-		(mirror x)
 		(unit 1)
 		(exclude_from_sim no)
@@
 		(dnp no)
 		(property "Reference" "D20"
-			(at 171.45 128.2699 90)
+			(at 171.45 130.8101 90)
 			(effects
 				(font
@@
 		)
 		(property "Value" "PTVS26VZ1USK"
-			(at 171.45 130.8099 90)
+			(at 171.45 128.2701 90)
 			(effects
 				(font
@@
 		(lib_id "Diode:PTVS26VZ1USK")
 		(at 88.9 87.63 270)
-		(mirror x)
 		(unit 1)
 		(exclude_from_sim no)
@@
 		(dnp no)
 		(property "Reference" "D13"
-			(at 86.36 86.3599 90)
+			(at 86.36 88.9001 90)
 			(effects
 				(font
@@
 		)
 		(property "Value" "PTVS26VZ1USK"
-			(at 86.36 88.8999 90)
+			(at 86.36 86.3601 90)
 			(effects
 				(font
@@
 		(lib_id "Diode:PTVS26VZ1USK")
 		(at 29.21 87.63 270)
-		(mirror x)
 		(unit 1)
 		(exclude_from_sim no)
@@
 		(dnp no)
 		(property "Reference" "D9"
-			(at 26.67 86.3599 90)
+			(at 26.67 88.9001 90)
 			(effects
 				(font
@@
 		)
 		(property "Value" "PTVS26VZ1USK"
-			(at 26.67 88.8999 90)
+			(at 26.67 86.3601 90)
 			(effects
 				(font
@@
 		(lib_id "Diode:PTVS26VZ1USK")
 		(at 58.42 87.63 270)
-		(mirror x)
 		(unit 1)
 		(exclude_from_sim no)
@@
 		(dnp no)
 		(property "Reference" "D11"
-			(at 55.88 86.3599 90)
+			(at 55.88 88.9001 90)
 			(effects
 				(font
@@
 		)
 		(property "Value" "PTVS26VZ1USK"
-			(at 55.88 88.8999 90)
+			(at 55.88 86.3601 90)
 			(effects
 				(font
@@
 		(lib_id "Diode:PTVS26VZ1USK")
 		(at 173.99 58.42 270)
-		(mirror x)
 		(unit 1)
 		(exclude_from_sim no)
@@
 		(dnp no)
 		(property "Reference" "D17"
-			(at 171.45 57.1499 90)
+			(at 171.45 59.6901 90)
 			(effects
 				(font
@@
 		)
 		(property "Value" "PTVS26VZ1USK"
-			(at 171.45 59.6899 90)
+			(at 171.45 57.1501 90)
 			(effects
 				(font
@@
 		(lib_id "Diode:PTVS26VZ1USK")
 		(at 116.84 87.63 270)
-		(mirror x)
 		(unit 1)
 		(exclude_from_sim no)
@@
 		(dnp no)
 		(property "Reference" "D15"
-			(at 114.3 86.3599 90)
+			(at 114.3 88.9001 90)
 			(effects
 				(font
@@
 		)
 		(property "Value" "PTVS26VZ1USK"
-			(at 114.3 88.8999 90)
+			(at 114.3 86.3601 90)
 			(effects
 				(font
@@
 		(lib_id "Diode:PTVS26VZ1USK")
 		(at 173.99 82.55 270)
-		(mirror x)
 		(unit 1)
 		(exclude_from_sim no)
@@
 		(dnp no)
 		(property "Reference" "D18"
-			(at 171.45 81.2799 90)
+			(at 171.45 83.8201 90)
 			(effects
 				(font
@@
 		)
 		(property "Value" "PTVS26VZ1USK"
-			(at 171.45 83.8199 90)
+			(at 171.45 81.2801 90)
 			(effects
 				(font
