File: HARDWARE/TeR_ECU/MICRO.kicad_sch (KiCad schematic)
At the start: 30 parts, among them J3 DEBUG, SW1 RST, SW2 BOOT0, U5 STM32F405VGTx, Y1 ECX-12R, Y2 ECS-250-20-33-CKM-TR

Commit message: Cool things
Parts:
- added R23, R24: 10k, symbol Device:R_Small
Connections:
- net +3.3V: now also R23.1, R24.1
- net SCL_1: now also R23.2
- net SDA_1: now also R24.2
Other:
- note added: "I2C_1"

Commit message: Quick changes, go to start layouting
Parts:
- added R42, R43: 10k, symbol Device:R_Small
- C17: renamed from C18; footprint (none) -> Capacitor_SMD:C_0603_1608Metric
- C19, C20, C21, C22, C23: footprint (none) -> Capacitor_SMD:C_0603_1608Metric
- C24: renamed from C13; footprint (none) -> Capacitor_SMD:C_0603_1608Metric
- C25: renamed from C24; footprint (none) -> Capacitor_SMD:C_0603_1608Metric
- C26: renamed from C25; footprint (none) -> Capacitor_SMD:C_0603_1608Metric
- C27: renamed from C14; footprint (none) -> Capacitor_SMD:C_0603_1608Metric
- C30: renamed from C15; footprint (none) -> Capacitor_SMD:C_0603_1608Metric
- C31: renamed from C16; footprint (none) -> Capacitor_SMD:C_0603_1608Metric
- C32: renamed from C28; footprint (none) -> Capacitor_SMD:C_0805_2012Metric
- C33: renamed from C29; footprint (none) -> Capacitor_SMD:C_0805_2012Metric
- renumbered R19 to R35, R20 to R36, R21 to R37, R22 to R38, R23 to R39, R24 to R40, R17 to R41, R18 to R44, U5 to U6
Connections:
- net +3.3V: now also R42.1, R43.1
- net UART_RX: now also U6.69 (PA10); no longer U6.24 (PA1)
- net UART_TX: now also U6.68 (PA9); no longer U6.23 (PA0)
- net IN_2: now reaches U6.1 (PE2)
- net IN_3: now reaches U6.2 (PE3)
- net ADC1_2: now reaches U6.25 (PA2)
- net ADC1_3: now reaches U6.26 (PA3)
- net OUT_0: now reaches U6.3 (PE4)
- net SPI1_MOSI: now reaches U6.32 (PA7)
- net OUT_3: now reaches U6.38 (PE7)
- net SC_EN: now reaches U6.39 (PE8)
- net OUT_1: now reaches U6.4 (PE5)
- net T1_CH1: now reaches U6.40 (PE9)
- net T1_CH2: now reaches U6.42 (PE11)
- net T1_CH3: now reaches U6.44 (PE13)
- net T1_CH4: now reaches U6.45 (PE14)
- net SCL_2: now reaches U6.47 (PB10)
- net SCL_2: now also R42.2
- net SDA_2: now reaches U6.48 (PB11)
- net SDA_2: now also R43.2
- net OUT_2: now reaches U6.5 (PE6)
- net IN_0: now reaches U6.97 (PE0)
- net IN_1: now reaches U6.98 (PE1)
- net BL renamed IMU_LED
- net BSPD_3V3 renamed SYS_LED
- net Horn renamed SPI2_MOSI
- net SDIO_CK: no longer names the net of U6.80 (PC12)
- net SDIO_CMD: no longer names the net of U6.83 (PD2)
- net SDIO_D0: no longer names the net of U6.65 (PC8)
- net SDIO_D1: no longer names the net of U6.66 (PC9)
- net SDIO_D2: no longer names the net of U6.78 (PC10)
- net SDIO_D3: no longer names the net of U6.79 (PC11)
- net TSMS_3V3 renamed ERR_LED
- new net ADC1_0: U6.23 (PA0)
- new net ADC1_1: U6.24 (PA1)
- no-connect marks 1 -> 45
Other:
- note added: "I2C_2"

Commit message: Began layout
Parts:
- C17: footprint Capacitor_SMD:C_0603_1608Metric -> Capacitor_SMD:C_1210_3225Metric
- C19, C20, C21, C22, C23, C25, C26: footprint Capacitor_SMD:C_0603_1608Metric -> Capacitor_SMD:C_0402_1005Metric
- R39, R40, R41, R42, R43, R44: footprint (none) -> Resistor_SMD:R_0603_1608Metric
Connections:
- net OSC_IN is gone; now on net HSE_OUT: U6.12 (PH0)
- no-connect marks 45 -> 44
Changed lines of the file:
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@@
 	)
 	(no_connect
-		(at 209.55 43.18)
-	)
-	(no_connect
 		(at 255.27 149.86)
 	)
@@
 	(wire
 		(pts
-			(xy 200.66 40.64) (xy 209.55 40.64)
-		)
-		(stroke
-			(width 0)
-			(type default)
-		)
-	)
-	(wire
-		(pts
 			(xy 93.98 34.29) (xy 93.98 26.67)
 		)
@@
 		)
 	)
+	(wire
+		(pts
+			(xy 200.66 40.64) (xy 209.55 40.64)
+		)
+		(stroke
+			(width 0)
+			(type default)
+		)
+	)
 	(rectangle
 		(start 12.7 71.12)
@@
 		)
 	)
+	(label "HSE_OUT"
+		(at 209.55 40.64 180)
+		(fields_autoplaced yes)
+		(effects
+			(font
+				(size 1.27 1.27)
+			)
+			(justify right bottom)
+		)
+	)
 	(label "SDA_2"
 		(at 133.35 95.25 0)
@@
 		)
 	)
-	(label "OSC_IN"
-		(at 200.66 40.64 0)
-		(fields_autoplaced yes)
-		(effects
-			(font
-				(size 1.27 1.27)
-			)
-			(justify left bottom)
-		)
-	)
 	(label "LSE_OUT"
 		(at 124.46 26.67 180)
@@
 			)
 		)
-		(property "Footprint" ""
+		(property "Footprint" "Resistor_SMD:R_0603_1608Metric"
 			(at 143.51 87.63 0)
 			(effects
@@
 			)
 		)
-		(property "Footprint" "Capacitor_SMD:C_0603_1608Metric"
+		(property "Footprint" "Capacitor_SMD:C_0402_1005Metric"
 			(at 70.8152 129.54 0)
 			(effects
@@
 			)
 		)
-		(property "Footprint" "Capacitor_SMD:C_0603_1608Metric"
+		(property "Footprint" "Capacitor_SMD:C_0402_1005Metric"
 			(at 97.4852 129.54 0)
 			(effects
@@
 			)
 		)
-		(property "Footprint" ""
+		(property "Footprint" "Resistor_SMD:R_0603_1608Metric"
 			(at 162.052 30.48 90)
 			(effects
@@
 			)
 		)
-		(property "Footprint" ""
+		(property "Footprint" "Resistor_SMD:R_0603_1608Metric"
 			(at 148.59 87.63 0)
 			(effects
@@
 			)
 		)
-		(property "Footprint" ""
+		(property "Footprint" "Resistor_SMD:R_0603_1608Metric"
 			(at 106.68 87.63 0)
 			(effects
@@
 			)
 		)
-		(property "Footprint" "Capacitor_SMD:C_0603_1608Metric"
+		(property "Footprint" "Capacitor_SMD:C_0402_1005Metric"
 			(at 58.1152 129.54 0)
 			(effects
@@
 			)
 		)
-		(property "Footprint" "Capacitor_SMD:C_0603_1608Metric"
+		(property "Footprint" "Capacitor_SMD:C_0402_1005Metric"
 			(at 32.7152 129.54 0)
 			(effects
@@
 			)
 		)
-		(property "Footprint" ""
+		(property "Footprint" "Resistor_SMD:R_0603_1608Metric"
 			(at 113.792 30.48 90)
 			(effects
@@
 			)
 		)
-		(property "Footprint" "Capacitor_SMD:C_0603_1608Metric"
+		(property "Footprint" "Capacitor_SMD:C_1210_3225Metric"
 			(at 20.0152 129.54 0)
 			(effects
@@
 			)
 		)
-		(property "Footprint" "Capacitor_SMD:C_0603_1608Metric"
+		(property "Footprint" "Capacitor_SMD:C_0402_1005Metric"
 			(at 110.1852 129.54 0)
 			(effects
@@
 			)
 		)
-		(property "Footprint" "Capacitor_SMD:C_0603_1608Metric"
+		(property "Footprint" "Capacitor_SMD:C_0402_1005Metric"
 			(at 83.5152 129.54 0)
 			(effects
@@
 			)
 		)
-		(property "Footprint" ""
+		(property "Footprint" "Resistor_SMD:R_0603_1608Metric"
 			(at 101.6 87.63 0)
 			(effects
@@
 			)
 		)
-		(property "Footprint" "Capacitor_SMD:C_0603_1608Metric"
+		(property "Footprint" "Capacitor_SMD:C_0402_1005Metric"
 			(at 45.4152 129.54 0)
 			(effects

Commit message: First layout prototype
Parts:
- removed R41, R44: 0R, Resistor_SMD:R_0603_1608Metric, symbol Device:R
- C19, C20, C21, C22, C23, C25, C26: footprint Capacitor_SMD:C_0402_1005Metric -> Capacitor_SMD:C_0603_1608Metric
Connections:
- net HSE_IN: now also U6.12 (PH0)
- net HSE_OUT: now also C31.1, U6.13 (PH1), Y2.3; no longer U6.12 (PH0)
- net LSE_IN: now also U6.8 (PC14)
- net LSE_OUT: now also C27.1, U6.9 (PC15), Y1.2
- no-connect marks 44 -> 42
Changed lines of the file:
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@@
 	)
 	(junction
-		(at 115.57 34.29)
-		(diameter 0)
-		(color 0 0 0 0)
-	)
-	(junction
 		(at 143.51 92.71)
 		(diameter 0)
@@
 	)
 	(junction
-		(at 163.83 34.29)
+		(at 31.75 121.92)
 		(diameter 0)
 		(color 0 0 0 0)
 	)
 	(junction
-		(at 31.75 121.92)
+		(at 115.57 34.29)
 		(diameter 0)
 		(color 0 0 0 0)
@@
 	)
 	(junction
+		(at 163.83 34.29)
+		(diameter 0)
+		(color 0 0 0 0)
+	)
+	(junction
 		(at 101.6 92.71)
 		(diameter 0)
@@
 	)
 	(no_connect
-		(at 255.27 149.86)
-	)
-	(no_connect
 		(at 209.55 127)
 	)
@@
 	)
 	(no_connect
-		(at 255.27 147.32)
-	)
-	(no_connect
 		(at 255.27 68.58)
 	)
@@
 	(wire
 		(pts
+			(xy 264.16 147.32) (xy 255.27 147.32)
+		)
+		(stroke
+			(width 0)
+			(type default)
+		)
+	)
+	(wire
+		(pts
 			(xy 62.23 43.18) (xy 48.26 43.18)
 		)
@@
 	(wire
 		(pts
+			(xy 115.57 26.67) (xy 115.57 34.29)
+		)
+		(stroke
+			(width 0)
+			(type default)
+		)
+	)
+	(wire
+		(pts
 			(xy 157.48 121.92) (xy 152.4 121.92)
 		)
@@
 	(wire
 		(pts
+			(xy 264.16 149.86) (xy 255.27 149.86)
+		)
+		(stroke
+			(width 0)
+			(type default)
+		)
+	)
+	(wire
+		(pts
 			(xy 133.35 92.71) (xy 143.51 92.71)
 		)
@@
 	(wire
 		(pts
+			(xy 163.83 34.29) (xy 163.83 26.67)
+		)
+		(stroke
+			(width 0)
+			(type default)
+		)
+	)
+	(wire
+		(pts
 			(xy 148.59 95.25) (xy 153.67 95.25)
 		)
@@
 	(wire
 		(pts
-			(xy 163.83 34.29) (xy 157.48 34.29)
+			(xy 157.48 34.29) (xy 163.83 34.29)
 		)
 		(stroke
@@
 	(wire
 		(pts
+			(xy 200.66 43.18) (xy 209.55 43.18)
+		)
+		(stroke
+			(width 0)
+			(type default)
+		)
+	)
+	(wire
+		(pts
 			(xy 143.51 90.17) (xy 143.51 92.71)
 		)
@@
 		)
 	)
-	(label "HSE_OUT"
-		(at 209.55 40.64 180)
+	(label "SDA_2"
+		(at 133.35 95.25 0)
 		(fields_autoplaced yes)
 		(effects
@@
 				(size 1.27 1.27)
 			)
-			(justify right bottom)
+			(justify left bottom)
 		)
 	)
-	(label "SDA_2"
-		(at 133.35 95.25 0)
+	(label "LSE_OUT"
+		(at 264.16 149.86 180)
 		(fields_autoplaced yes)
 		(effects
@@
 				(size 1.27 1.27)
 			)
-			(justify left bottom)
+			(justify right bottom)
 		)
 	)
@@
 	)
 	(label "HSE_IN"
+		(at 200.66 40.64 0)
+		(fields_autoplaced yes)
+		(effects
+			(font
+				(size 1.27 1.27)
+			)
+			(justify left bottom)
+		)
+	)
+	(label "HSE_IN"
 		(at 135.89 26.67 0)
 		(fields_autoplaced yes)
@@
 		)
 	)
+	(label "HSE_OUT"
+		(at 200.66 43.18 0)
+		(fields_autoplaced yes)
+		(effects
+			(font
+				(size 1.27 1.27)
+			)
+			(justify left bottom)
+		)
+	)
 	(label "SCL_1"
 		(at 265.43 83.82 180)
@@
 		)
 	)
+	(label "LSE_IN"
+		(at 264.16 147.32 180)
+		(fields_autoplaced yes)
+		(effects
+			(font
+				(size 1.27 1.27)
+			)
+			(justify right bottom)
+		)
+	)
 	(label "SCL_2"
 		(at 133.35 92.71 0)
@@
 			)
 		)
-		(property "Footprint" "Capacitor_SMD:C_0402_1005Metric"
+		(property "Footprint" "Capacitor_SMD:C_0603_1608Metric"
 			(at 70.8152 129.54 0)
 			(effects
@@
 			)
 		)
-		(property "Footprint" "Capacitor_SMD:C_0402_1005Metric"
+		(property "Footprint" "Capacitor_SMD:C_0603_1608Metric"
 			(at 97.4852 129.54 0)
 			(effects
@@
 	)
 	(symbol
-		(lib_id "Device:R")
-		(at 163.83 30.48 0)
-		(unit 1)
-		(exclude_from_sim no)
-		(in_bom yes)
-		(on_board yes)
-		(dnp no)
-		(fields_autoplaced yes)
-		(property "Reference" "R44"
-			(at 166.37 29.2099 0)
-			(effects
-				(font
-					(size 1.27 1.27)
-				)
-				(justify left)
-			)
-		)
-		(property "Value" "0R"
-			(at 166.37 31.7499 0)
-			(effects
-				(font
-					(size 1.27 1.27)
-				)
-				(justify left)
-			)
-		)
-		(property "Footprint" "Resistor_SMD:R_0603_1608Metric"
-			(at 162.052 30.48 90)
-			(effects
-				(font
-					(size 1.27 1.27)
-				)
-				(hide yes)
-			)
-		)
-		(property "Datasheet" "~"
-			(at 163.83 30.48 0)
-			(effects
-				(font
-					(size 1.27 1.27)
-				)
-				(hide yes)
-			)
-		)
-		(property "Description" "Resistor"
-			(at 163.83 30.48 0)
-			(effects
-				(font
-					(size 1.27 1.27)
-				)
-				(hide yes)
-			)
-		)
-		(pin "2"
-		)
-		(pin "1"
-		)
-		(instances
-			(project "TeR_ECU"
-				(path "/84413845-c4f3-4743-bcd2-a67649c90902/6cf54a6a-28e2-462f-b0c6-d7147ca367a6"
-					(reference "R44")
-					(unit 1)
-				)
-			)
-		)
-	)
-	(symbol
 		(lib_name "GND_1")
 		(lib_id "power:GND")
@@
 			)
 		)
-		(property "Footprint" "Capacitor_SMD:C_0402_1005Metric"
+		(property "Footprint" "Capacitor_SMD:C_0603_1608Metric"
 			(at 58.1152 129.54 0)
 			(effects
@@
 			)
 		)
-		(property "Footprint" "Capacitor_SMD:C_0402_1005Metric"
+		(property "Footprint" "Capacitor_SMD:C_0603_1608Metric"
 			(at 32.7152 129.54 0)
 			(effects
@@
 	)
 	(symbol
-		(lib_id "Device:R")
-		(at 115.57 30.48 0)
-		(unit 1)
-		(exclude_from_sim no)
-		(in_bom yes)
-		(on_board yes)
-		(dnp no)
-		(fields_autoplaced yes)
-		(property "Reference" "R41"
-			(at 118.11 29.2099 0)
-			(effects
-				(font
-					(size 1.27 1.27)
-				)
-				(justify left)
-			)
-		)
-		(property "Value" "0R"
-			(at 118.11 31.7499 0)
-			(effects
-				(font
-					(size 1.27 1.27)
-				)
-				(justify left)
-			)
-		)
-		(property "Footprint" "Resistor_SMD:R_0603_1608Metric"
-			(at 113.792 30.48 90)
-			(effects
-				(font
-					(size 1.27 1.27)
-				)
-				(hide yes)
-			)
-		)
-		(property "Datasheet" "~"
-			(at 115.57 30.48 0)
-			(effects
-				(font
-					(size 1.27 1.27)
-				)
-				(hide yes)
-			)
-		)
-		(property "Description" "Resistor"
-			(at 115.57 30.48 0)
-			(effects
-				(font
-					(size 1.27 1.27)
-				)
-				(hide yes)
-			)
-		)
-		(pin "2"
-		)
-		(pin "1"
-		)
-		(instances
-			(project "TeR_ECU"
-				(path "/84413845-c4f3-4743-bcd2-a67649c90902/6cf54a6a-28e2-462f-b0c6-d7147ca367a6"
-					(reference "R41")
-					(unit 1)
-				)
-			)
-		)
-	)
-	(symbol
 		(lib_id "Device:C")
 		(at 19.05 125.73 0)
@@
 			)
 		)
-		(property "Footprint" "Capacitor_SMD:C_0402_1005Metric"
+		(property "Footprint" "Capacitor_SMD:C_0603_1608Metric"
 			(at 110.1852 129.54 0)
 			(effects
@@
 			)
 		)
-		(property "Footprint" "Capacitor_SMD:C_0402_1005Metric"
+		(property "Footprint" "Capacitor_SMD:C_0603_1608Metric"
 			(at 83.5152 129.54 0)
 			(effects
@@
 			)
 		)
-		(property "Footprint" "Capacitor_SMD:C_0402_1005Metric"
+		(property "Footprint" "Capacitor_SMD:C_0603_1608Metric"
 			(at 45.4152 129.54 0)
 			(effects

Commit message: Finished layout, RF design, and quick DRC check, Lookin gud
Connections:
- net ADC1_0: now also U6.25 (PA2); no longer U6.23 (PA0)
- net ADC1_1: now also U6.26 (PA3); no longer U6.24 (PA1)
- net ADC1_2: now also U6.23 (PA0); no longer U6.25 (PA2)
- net ADC1_3: now also U6.24 (PA1); no longer U6.26 (PA3)
- net ERR_LED: now also U6.36 (PB1); no longer U6.16 (PC1)
- net IMU_LED: now also U6.37 (PB2); no longer U6.17 (PC2)
- net IN_0: now also U6.5 (PE6); no longer U6.97 (PE0)
- net IN_1: now also U6.4 (PE5); no longer U6.98 (PE1)
- net IN_2: now also U6.3 (PE4); no longer U6.1 (PE2)
- net IN_3: now also U6.38 (PE7); no longer U6.2 (PE3)
- net OUT_0: now also U6.2 (PE3); no longer U6.3 (PE4)
- net OUT_1: now also U6.1 (PE2); no longer U6.4 (PE5)
- net OUT_2: now also U6.98 (PE1); no longer U6.5 (PE6)
- net OUT_3: now also U6.97 (PE0); no longer U6.38 (PE7)
- net SC_EN: now also U6.96 (PB9); no longer U6.39 (PE8)
- net SYS_LED: now also U6.35 (PB0); no longer U6.15 (PC0)
- net T3_CH1: now reaches U6.63 (PC6)
- net T3_CH2: now reaches U6.64 (PC7)
- net T3_CH3: now reaches U6.65 (PC8)
- net T3_CH4: now reaches U6.66 (PC9)
- net T1_CH1: no longer names the net of U6.40 (PE9)
- net T1_CH2: no longer names the net of U6.42 (PE11)
- net T1_CH3: no longer names the net of U6.44 (PE13)
- net T1_CH4: no longer names the net of U6.45 (PE14)
