File: HARDWARE/TeR_ECU/MICRO.kicad_sch (KiCad schematic)
At the start: 32 parts, among them J3 DEBUG, SW1 RST, SW2 BOOT0, U6 STM32F405VGTx, Y1 ECX-12R, Y2 ECS-250-20-33-CKM-TR

Commit message: Corregidos conectores, CAN y añadidas librerias al proyecto para cargar huellas
Parts:
- renumbered C14 to C18, C1 to C28, C5 to C29
