File: HARDWARE/TeR_ECU/WS2812.kicad_sch (KiCad schematic)
At the start: 2 parts

Commit message: Quick changes, go to start layouting
Parts:
- added D6: SMAJ6.0A, Diode_SMD:D_SMA, symbol Diode:SMAJ6.0A
- added R6: 100R, symbol Device:R
- renumbered D19 to D5, R25 to R5
Connections:
- net GND: now also D6.1 (A1)
- net LED_DATA renamed LED1
- net LED_SPI renamed LED1_SPI
- new net LED2: D6.2 (A2), R6.1
- new net LED2_SPI: R6.2
Other:
- moved on the sheet: D5, R5

Commit message: Began layout
Parts:
- removed D5, D6: SMAJ6.0A, Diode_SMD:D_SMA, symbol Diode:SMAJ6.0A
- added D32, D5: PTVS7V5Z1USK, Diode_SMD:Nexperia_DSN1608-2_1.6x0.8mm, symbol Diode:PTVS7V5Z1USK
- R5, R6: footprint (none) -> Resistor_SMD:R_0603_1608Metric
Connections:
- net GND: now also D32.1 (K), D5.1 (K)
- net LED1: now also D32.2 (A)
- net LED2: now also D5.2 (A)
Changed lines of the file:
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@@
+	)
+	(junction
+		(at 130.81 87.63)
+		(diameter 0)
+		(color 0 0 0 0)
 	)
 	(junction
@@
 		(color 0 0 0 0)
 	)
-	(junction
-		(at 130.81 87.63)
-		(diameter 0)
-		(color 0 0 0 0)
+	(wire
+		(pts
+			(xy 130.81 87.63) (xy 140.97 87.63)
+		)
+		(stroke
+			(width 0)
+			(type default)
+		)
 	)
 	(wire
@@
 	(wire
 		(pts
+			(xy 120.65 67.31) (xy 130.81 67.31)
+		)
+		(stroke
+			(width 0)
+			(type default)
+		)
+	)
+	(wire
+		(pts
+			(xy 148.59 87.63) (xy 163.83 87.63)
+		)
+		(stroke
+			(width 0)
+			(type default)
+		)
+	)
+	(wire
+		(pts
 			(xy 130.81 67.31) (xy 140.97 67.31)
-		)
-		(stroke
-			(width 0)
-			(type default)
-		)
-	)
-	(wire
-		(pts
-			(xy 120.65 67.31) (xy 130.81 67.31)
-		)
-		(stroke
-			(width 0)
-			(type default)
-		)
-	)
-	(wire
-		(pts
-			(xy 130.81 87.63) (xy 140.97 87.63)
-		)
-		(stroke
-			(width 0)
-			(type default)
-		)
-	)
-	(wire
-		(pts
-			(xy 148.59 87.63) (xy 163.83 87.63)
 		)
 		(stroke
@@
 	)
 	(symbol
-		(lib_id "Diode:SMAJ6.0A")
-		(at 130.81 71.12 90)
+		(lib_id "Diode:PTVS7V5Z1USK")
+		(at 130.81 91.44 90)
 		(unit 1)
 		(exclude_from_sim no)
@@
 		(fields_autoplaced yes)
 		(property "Reference" "D5"
+			(at 133.35 90.1699 90)
+			(effects
+				(font
+					(size 1.27 1.27)
+				)
+				(justify right)
+			)
+		)
+		(property "Value" "PTVS7V5Z1USK"
+			(at 133.35 92.7099 90)
+			(effects
+				(font
+					(size 1.27 1.27)
+				)
+				(justify right)
+			)
+		)
+		(property "Footprint" "Diode_SMD:Nexperia_DSN1608-2_1.6x0.8mm"
+			(at 135.255 91.44 0)
+			(effects
+				(font
+					(size 1.27 1.27)
+				)
+				(hide yes)
+			)
+		)
+		(property "Datasheet" "https://assets.nexperia.com/documents/data-sheet/PTVS7V5Z1USK.pdf"
+			(at 130.81 91.44 0)
+			(effects
+				(font
+					(size 1.27 1.27)
+				)
+				(hide yes)
+			)
+		)
+		(property "Description" "7.5V, 2200W TVS unidirectional diode, DSN1608-2"
+			(at 130.81 91.44 0)
+			(effects
+				(font
+					(size 1.27 1.27)
+				)
+				(hide yes)
+			)
+		)
+		(pin "2"
+		)
+		(pin "1"
+		)
+		(instances
+			(project "TeR_ECU"
+				(path "/84413845-c4f3-4743-bcd2-a67649c90902/57c564d0-e71b-4ec8-8e08-7691aefb5091"
+					(reference "D5")
+					(unit 1)
+				)
+			)
+		)
+	)
+	(symbol
+		(lib_id "Diode:PTVS7V5Z1USK")
+		(at 130.81 71.12 90)
+		(unit 1)
+		(exclude_from_sim no)
+		(in_bom yes)
+		(on_board yes)
+		(dnp no)
+		(fields_autoplaced yes)
+		(property "Reference" "D32"
 			(at 133.35 69.8499 90)
 			(effects
@@
 			)
 		)
-		(property "Value" "SMAJ6.0A"
+		(property "Value" "PTVS7V5Z1USK"
 			(at 133.35 72.3899 90)
 			(effects
@@
 			)
 		)
-		(property "Footprint" "Diode_SMD:D_SMA"
-			(at 135.89 71.12 0)
-			(effects
-				(font
-					(size 1.27 1.27)
-				)
-				(hide yes)
-			)
-		)
-		(property "Datasheet" "https://www.littelfuse.com/media?resourcetype=datasheets&itemid=75e32973-b177-4ee3-a0ff-cedaf1abdb93&filename=smaj-datasheet"
-			(at 130.81 72.39 0)
-			(effects
-				(font
-					(size 1.27 1.27)
-				)
-				(hide yes)
-			)
-		)
-		(property "Description" "400W unidirectional Transient Voltage Suppressor, 6.0Vr, SMA(DO-214AC)"
+		(property "Footprint" "Diode_SMD:Nexperia_DSN1608-2_1.6x0.8mm"
+			(at 135.255 71.12 0)
+			(effects
+				(font
+					(size 1.27 1.27)
+				)
+				(hide yes)
+			)
+		)
+		(property "Datasheet" "https://assets.nexperia.com/documents/data-sheet/PTVS7V5Z1USK.pdf"
+			(at 130.81 71.12 0)
+			(effects
+				(font
+					(size 1.27 1.27)
+				)
+				(hide yes)
+			)
+		)
+		(property "Description" "7.5V, 2200W TVS unidirectional diode, DSN1608-2"
 			(at 130.81 71.12 0)
 			(effects
@@
 			(project ""
 				(path "/84413845-c4f3-4743-bcd2-a67649c90902/57c564d0-e71b-4ec8-8e08-7691aefb5091"
-					(reference "D5")
-					(unit 1)
-				)
-			)
-		)
-	)
-	(symbol
-		(lib_id "Diode:SMAJ6.0A")
-		(at 130.81 91.44 90)
-		(unit 1)
-		(exclude_from_sim no)
-		(in_bom yes)
-		(on_board yes)
-		(dnp no)
-		(fields_autoplaced yes)
-		(property "Reference" "D6"
-			(at 133.35 90.1699 90)
-			(effects
-				(font
-					(size 1.27 1.27)
-				)
-				(justify right)
-			)
-		)
-		(property "Value" "SMAJ6.0A"
-			(at 133.35 92.7099 90)
-			(effects
-				(font
-					(size 1.27 1.27)
-				)
-				(justify right)
-			)
-		)
-		(property "Footprint" "Diode_SMD:D_SMA"
-			(at 135.89 91.44 0)
-			(effects
-				(font
-					(size 1.27 1.27)
-				)
-				(hide yes)
-			)
-		)
-		(property "Datasheet" "https://www.littelfuse.com/media?resourcetype=datasheets&itemid=75e32973-b177-4ee3-a0ff-cedaf1abdb93&filename=smaj-datasheet"
-			(at 130.81 92.71 0)
-			(effects
-				(font
-					(size 1.27 1.27)
-				)
-				(hide yes)
-			)
-		)
-		(property "Description" "400W unidirectional Transient Voltage Suppressor, 6.0Vr, SMA(DO-214AC)"
-			(at 130.81 91.44 0)
-			(effects
-				(font
-					(size 1.27 1.27)
-				)
-				(hide yes)
-			)
-		)
-		(pin "2"
-		)
-		(pin "1"
-		)
-		(instances
-			(project "TeR_ECU"
-				(path "/84413845-c4f3-4743-bcd2-a67649c90902/57c564d0-e71b-4ec8-8e08-7691aefb5091"
-					(reference "D6")
+					(reference "D32")
 					(unit 1)
 				)
@@
 			)
 		)
-		(property "Footprint" ""
+		(property "Footprint" "Resistor_SMD:R_0603_1608Metric"
 			(at 144.78 69.088 90)
 			(effects
@@
 			)
 		)
-		(property "Footprint" ""
+		(property "Footprint" "Resistor_SMD:R_0603_1608Metric"
 			(at 144.78 89.408 90)
 			(effects

Commit message: Finished layout, RF design, and quick DRC check, Lookin gud
Connections:
- net GND: now also D32.2 (A), D5.2 (A); no longer D32.1 (K), D5.1 (K)
- net LED1: now also D32.1 (K); no longer D32.2 (A)
- net LED2: now also D5.1 (K); no longer D5.2 (A)
Changed lines of the file:
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@@
 		(lib_id "Diode:PTVS7V5Z1USK")
 		(at 130.81 91.44 90)
+		(mirror x)
 		(unit 1)
 		(exclude_from_sim no)
@@
 		(on_board yes)
 		(dnp no)
-		(fields_autoplaced yes)
 		(property "Reference" "D5"
-			(at 133.35 90.1699 90)
+			(at 133.35 92.7101 90)
 			(effects
 				(font
@@
 		)
 		(property "Value" "PTVS7V5Z1USK"
-			(at 133.35 92.7099 90)
+			(at 133.35 90.1701 90)
 			(effects
 				(font
@@
 		(lib_id "Diode:PTVS7V5Z1USK")
 		(at 130.81 71.12 90)
+		(mirror x)
 		(unit 1)
 		(exclude_from_sim no)
@@
 		(on_board yes)
 		(dnp no)
-		(fields_autoplaced yes)
 		(property "Reference" "D32"
-			(at 133.35 69.8499 90)
+			(at 133.35 72.3901 90)
 			(effects
 				(font
@@
 		)
 		(property "Value" "PTVS7V5Z1USK"
-			(at 133.35 72.3899 90)
+			(at 133.35 69.8501 90)
 			(effects
 				(font
