File: HARDWARE/TeR_ECU/CAN.kicad_sch (KiCad schematic)
At the start: 10 parts, among them U5 TCAN332

Commit message: abrirlo en kicad y q funcione
Parts:
- renumbered C17 to C1, C32 to C2, C18 to C3, C22 to C4, D2 to D7, FL2 to FL1, JP2 to JP1, R9 to R7, R32 to R8, U5 to U1
