File: HARDWARE/TeR_ECU/CAN.kicad_sch (KiCad schematic)
At the start: 10 parts, among them U5 TCAN332

Commit message: Corregidos conectores, CAN y añadidas librerias al proyecto para cargar huellas
Parts:
- removed FL2: ACT45B-510-2P-TL003, CAN_CMF:FIL_ACT45B-510-2P-TL003, symbol CAN_CMF:ACT45B-510-2P-TL003
- removed JP2: 120R Term, Jumper:SolderJumper-3_P1.3mm_Open_RoundedPad1.0x1.5mm, symbol Jumper:SolderJumper_3_Open
- removed U5: TCAN332, Package_SO:SOIC-8_3.9x4.9mm_P1.27mm, symbol Interface_CAN_LIN:TCAN332
- added C41: 100n, Capacitor_SMD:C_0603_1608Metric, symbol Device:C_Small
- added FL1: ACT45B-510-2P-TL003, ACT45B-510-2P-TL003:ACT45B1012PTL003, symbol ACT45B-510-2P-TL003:ACT45B-510-2P-TL003
- added JP1: SolderJumper_3_Open, Jumper:SolderJumper-3_P1.3mm_Open_Pad1.0x1.5mm, symbol Jumper:SolderJumper_3_Open
- added U1: TCAN3403DR-Q1, Package_SO:SOIC-8_3.9x4.9mm_P1.27mm, symbol Interface_CAN_LIN:TCAN332
- renumbered C17 to C1, C32 to C2, C18 to C3, C22 to C4, D2 to D7, R9 to R7, R32 to R8
Connections:
- net +3.3V: now also C41.1, U1.3 (VCC), U1.5 (SHDNVIO)
- net CAN+: now also FL1.2
- net CAN-: now also FL1.1
- net CAN_RX: now also U1.4 (RXD)
- net CAN_TX: now also U1.1 (TXD)
- net GND: now also C41.2, U1.2 (GND), U1.8 (STB)
- net at R7.2: now also JP1.1 (A)
- net at C2.1: now also JP1.2 (C)
- net at R8.1: now also JP1.3 (B)
- net at D7.1 (K): now also FL1.4, U1.6 (CANL)
- net at D7.2 (K): now also FL1.3, U1.7 (CANH)
Other:
- note added: "Actualizado"
- note added: "Actualizado. Modificar a C5 y C9 o se deja en C41 y C43?"
