File: HARDWARE/TeR_ECU/POWER.kicad_sch (KiCad schematic)
At the start: 8 parts, among them U10 LM1117MP-3.3, U2 TSR_1-2450

Commit message: abrirlo en kicad y q funcione
Parts:
- renumbered C23 to C11, C24 to C12, U2 to U3, U10 to U4
