File: HARDWARE/TeR_ECU/POWER.kicad_sch (KiCad schematic)
At the start: 8 parts, among them U10 LM1117MP-3.3, U2 TSR_1-2450

Commit message: Corregidos conectores, CAN y añadidas librerias al proyecto para cargar huellas
Parts:
- L1: footprint footprints:IND_TCK-141_TRP -> Inductor_SMD:L_TracoPower_TCK-141
- renumbered C23 to C11, C24 to C12, U2 to U3, U10 to U4
