File: HARDWARE/TeR_ECU/RELAY.kicad_sch (KiCad schematic)
At the start: 5 parts, among them K2 G5Q-1, Q1 ZXMN3F30FH

Commit message: abrirlo en kicad y q funcione
Parts:
- renumbered Q1 to Q5, R28 to R51, R27 to R52
